Commit message: kuka demo update

File: kuka_description/lbr5_7.urdf (robot description, URDF)
Before this commit: robot lbr5_7, 9 links, 8 joints
Links:
- added link goal_1_link
- added link goal_2_link
- added link goal_3_link
- added link goal_4_link
- added link goal_5_link
- added link goal_6_link
- added link kuka_root; visual box size=0.001 0.001 0.001
- added link tcp_1_link
- added link tcp_2_link
- added link tool; collision mesh filename=package://kuka_description/cad/tool_s.dae; visual mesh filename=package://kuka_description/cad/tool_s.dae
Joints:
- added joint joint_goal_1: type fixed, parent kuka_root, child goal_1_link, origin xyz=2.0 0.5 12.0 rpy=-1.570796 0 1.570796, axis 0 0 1
- added joint joint_goal_2: type fixed, parent kuka_root, child goal_2_link, origin xyz=2.0 1.0 12.0 rpy=-1.570796 0 1.570796, axis 0 0 1
- added joint joint_goal_3: type fixed, parent kuka_root, child goal_3_link, origin xyz=2.0 1.5 12.0 rpy=-1.570796 0 1.570796, axis 0 0 1
- added joint joint_goal_4: type fixed, parent kuka_root, child goal_4_link, origin xyz=2.0 2.0 8.5 rpy=-1.570796 0 3.141592, axis 0 0 1
- added joint joint_goal_5: type fixed, parent kuka_root, child goal_5_link, origin xyz=1.5 2.0 8.5 rpy=-1.570796 0 3.141592, axis 0 0 1
- added joint joint_goal_6: type fixed, parent kuka_root, child goal_6_link, origin xyz=1.0 2.0 8.5 rpy=-1.570796 0 3.141592, axis 0 0 1
- added joint joint_root: type fixed, parent kuka_root, child segment_0, origin xyz=5.4 1.9 4.16 rpy=0 0 3.14159, axis 0 0 1
- added joint joint_tcp_1: type fixed, parent tool, child tcp_1_link, origin xyz=-1.64 -0.28 2.32, axis 0 0 1
- added joint joint_tcp_2: type fixed, parent tool, child tcp_2_link, origin xyz=-2.94 -0.11 0.44 rpy=0 -1.570796 0, axis 0 0 1
- added joint joint_tool: type fixed, parent segment_7, child tool, origin xyz=0 0 0, axis 0 0 1
- joint joint_ee: origin xyz=0 0 0.25 -> xyz=0 0 0; parent segment_7 -> tool
