Commit message: add collision meshes

File: human_description/robots/human_cio.urdf.xacro (robot description, xacro)
@@ -140,5 +140,5 @@
       <origin rpy="0 0 0" xyz="0 0 0"/>
       <geometry>
-        <mesh filename="package://human_description/meshes/pelvis.dae"/>
+        <mesh filename="package://human_description/meshes/collision/pelvis.dae"/>
       </geometry>
     </collision>
@@ -183,5 +183,5 @@
       <origin rpy="0 0 0" xyz="0 0 0"/>
       <geometry>
-        <mesh filename="package://human_description/meshes/torso.dae"/>
+        <mesh filename="package://human_description/meshes/collision/torso.dae"/>
       </geometry>
     </collision>
@@ -226,5 +226,5 @@
       <origin rpy="0 0 0" xyz="0 0 0"/>
       <geometry>
-        <mesh filename="package://human_description/meshes/head.dae"/>
+        <mesh filename="package://human_description/meshes/collision/head.dae"/>
       </geometry>
     </collision>
@@ -295,5 +295,5 @@
       <origin rpy="0 0 0" xyz="0 0 0"/>
       <geometry>
-        <mesh filename="package://human_description/meshes/upperLeftLeg.dae"/>
+        <mesh filename="package://human_description/meshes/collision/upperLeftLeg.dae"/>
       </geometry>
     </collision>
@@ -322,5 +322,5 @@
       <origin rpy="0 0 0" xyz="0 0 0"/>
       <geometry>
-        <mesh filename="package://human_description/meshes/lowerLeftLeg.dae"/>
+        <mesh filename="package://human_description/meshes/collision/lowerLeftLeg.dae"/>
       </geometry>
     </collision>
@@ -368,5 +368,5 @@
       <origin rpy="0 0 0" xyz="0 0 0"/>
       <geometry>
-        <mesh filename="package://human_description/meshes/leftFoot.dae"/>
+        <mesh filename="package://human_description/meshes/collision/leftFoot.dae"/>
       </geometry>
     </collision>
@@ -431,5 +431,5 @@
       <origin rpy="0 0 0" xyz="0 0 0"/>
       <geometry>
-        <mesh filename="package://human_description/meshes/upperRightLeg.dae"/>
+        <mesh filename="package://human_description/meshes/collision/upperRightLeg.dae"/>
       </geometry>
     </collision>
@@ -458,5 +458,5 @@
       <origin rpy="0 0 0" xyz="0 0 0"/>
       <geometry>
-        <mesh filename="package://human_description/meshes/lowerRightLeg.dae"/>
+        <mesh filename="package://human_description/meshes/collision/lowerRightLeg.dae"/>
       </geometry>
     </collision>
@@ -504,5 +504,5 @@
       <origin rpy="0 0 0" xyz="0 0 0"/>
       <geometry>
-        <mesh filename="package://human_description/meshes/rightFoot.dae"/>
+        <mesh filename="package://human_description/meshes/collision/rightFoot.dae"/>
       </geometry>
     </collision>
@@ -563,5 +563,5 @@
       <origin rpy="0 0 0" xyz="0 0 0"/>
       <geometry>
-        <mesh filename="package://human_description/meshes/upperLeftArm.dae"/>
+        <mesh filename="package://human_description/meshes/collision/upperLeftArm.dae"/>
       </geometry>
     </collision>
@@ -590,5 +590,5 @@
       <origin rpy="0 0 0" xyz="0 0 0"/>
       <geometry>
-        <mesh filename="package://human_description/meshes/lowerLeftArm.dae"/>
+        <mesh filename="package://human_description/meshes/collision/lowerLeftArm.dae"/>
       </geometry>
     </collision>
@@ -633,5 +633,5 @@
       <origin rpy="0 1.57 -1.57" xyz="0 0 0"/>
       <geometry>
-        <mesh filename="package://human_description/meshes/leftHand.dae"/>
+        <mesh filename="package://human_description/meshes/collision/leftHand.dae"/>
       </geometry>
     </collision>
@@ -698,5 +698,5 @@
       <origin rpy="0 0 0" xyz="0 0 0"/>
       <geometry>
-        <mesh filename="package://human_description/meshes/upperRightArm.dae"/>
+        <mesh filename="package://human_description/meshes/collision/upperRightArm.dae"/>
       </geometry>
     </collision>
@@ -725,5 +725,5 @@
       <origin rpy="0 0 0" xyz="0 0 0"/>
       <geometry>
-        <mesh filename="package://human_description/meshes/lowerRightArm.dae"/>
+        <mesh filename="package://human_description/meshes/collision/lowerRightArm.dae"/>
       </geometry>
     </collision>
@@ -768,5 +768,5 @@
       <origin rpy="0 -1.57 1.57" xyz="0 0 0"/>
       <geometry>
-        <mesh filename="package://human_description/meshes/rightHand.dae"/>
+        <mesh filename="package://human_description/meshes/collision/rightHand.dae"/>
       </geometry>
     </collision>

Commit message: ftr as cost function penalizing too much force in contacts, not converging

File: human_description/robots/human_cio.urdf.xacro (robot description, xacro)
@@ -97,6 +97,6 @@
   <joint name="base_prismatic_joint_z" type="prismatic">
     <axis xyz="0 0 1"/>
-    <limit effort="10000" lower="-1.12" upper="0.6" velocity="0.6"/>
-    <safety_controller k_position="100" k_velocity="2000000" soft_lower_limit="-1.1" soft_upper_limit="0.6"/>
+    <limit effort="10000" lower="-10.0" upper="10.0" velocity="0.6"/>
+    <safety_controller k_position="100" k_velocity="2000000" soft_lower_limit="-10.0" soft_upper_limit="10.0"/>
     <calibration falling="0.00536"/>
     <dynamics damping="20000.0"/>

Commit message: door opening

File: human_description/robots/human_cio.urdf.xacro (robot description, xacro)
@@ -799,3 +799,23 @@
     </collision>
   </link>
+  <link name="right_hand_door_link">
+    <visual>
+      <origin rpy="0 0 0" xyz="0.5 0.065 -1.6"/>
+      <geometry>
+        <mesh filename="package://move_itomp/meshes/door.dae"/>
+      </geometry>
+      <material name="Blue"/>
+    </visual>
+    <collision>
+      <origin rpy="0 0 0" xyz="0.5 0.065 -1.6"/>
+      <geometry>
+        <box size="0.001 0.001 0.001"/>
+      </geometry>
+    </collision>
+  </link>
+  <joint name="door_joint" type="fixed">
+    <origin rpy="-1.57 0 0" xyz="0 0 0"/>
+    <parent link="right_hand_endeffector_link"/>
+    <child link="right_hand_door_link"/>
+  </joint>
 </robot>

Commit message: update human_cio description for Humanoid14

File: human_description/robots/human_cio.urdf.xacro (robot description, xacro)
@@ -105,16 +105,14 @@
     <child link="base_prismatic_dummy3"/>
   </joint>
-  <joint name="base_revolute_joint_x" type="continuous">
-<!--  <joint name="base_revolute_joint_x" type="revolute">-->
-<!--    <limit effort="15" lower="-1.57079632679" upper="1.57079632679" velocity="5"/>-->
-    <axis xyz="1 0 0"/>
+  <joint name="base_revolute_joint_x" type="revolute">
+    <axis xyz="1 0 0"/>
+    <limit effort="15" lower="0.0" upper="0.0" velocity="5"/>
     <origin rpy="0 0 0" xyz="0 0 0"/>
     <parent link="base_prismatic_dummy3"/>
     <child link="base_revolute_dummy1"/>
   </joint>
-  <joint name="base_revolute_joint_y" type="continuous">
-<!--  <joint name="base_revolute_joint_y" type="revolute">-->
-<!--    <limit effort="15" lower="-1.57079632679" upper="1.57079632679" velocity="5"/>-->
-    <axis xyz="0 1 0"/>
+  <joint name="base_revolute_joint_y" type="revolute">
+    <axis xyz="0 1 0"/>
+    <limit effort="15" lower="0.0" upper="0.0" velocity="5"/>
     <origin rpy="0 0 0" xyz="0 0 0"/>
     <parent link="base_revolute_dummy1"/>
@@ -122,6 +120,4 @@
   </joint>
   <joint name="base_revolute_joint_z" type="continuous">
-<!--  <joint name="base_revolute_joint_z" type="revolute">-->
-<!--    <limit effort="15" lower="-1.57079632679" upper="1.57079632679" velocity="5"/>-->
     <axis xyz="0 0 1"/>
     <origin rpy="0 0 0" xyz="0 0 0"/>
@@ -624,5 +620,6 @@
   <link name="left_hand_x_link">
     <visual>
-      <origin rpy="0 1.57 -1.57" xyz="0 0 0"/>
+<!--      <origin rpy="0 1.57 -1.57" xyz="0 0 0"/>-->
+      <origin rpy="0 0 0" xyz="0 0 0"/>
       <geometry>
         <mesh filename="package://human_description/meshes/leftHand.dae"/>
@@ -631,5 +628,6 @@
     </visual>
     <collision>
-      <origin rpy="0 1.57 -1.57" xyz="0 0 0"/>
+<!--      <origin rpy="0 1.57 -1.57" xyz="0 0 0"/>-->
+      <origin rpy="0 0 0" xyz="0 0 0"/>
       <geometry>
         <mesh filename="package://human_description/meshes/collision/leftHand.dae"/>
@@ -759,5 +757,6 @@
   <link name="right_hand_x_link">
     <visual>
-      <origin rpy="0 -1.57 1.57" xyz="0 0 0"/>
+<!--      <origin rpy="0 -1.57 1.57" xyz="0 0 0"/>-->
+      <origin rpy="0 0 0" xyz="0 0 0"/>
       <geometry>
         <mesh filename="package://human_description/meshes/rightHand.dae"/>
@@ -766,5 +765,6 @@
     </visual>
     <collision>
-      <origin rpy="0 -1.57 1.57" xyz="0 0 0"/>
+<!--      <origin rpy="0 -1.57 1.57" xyz="0 0 0"/>-->
+      <origin rpy="0 0 0" xyz="0 0 0"/>
       <geometry>
         <mesh filename="package://human_description/meshes/collision/rightHand.dae"/>
@@ -799,5 +799,6 @@
     </collision>
   </link>
-  <link name="right_hand_door_link">
+<!--
+  <link name="right_hand_object_link">
     <visual>
       <origin rpy="0 0 0" xyz="0.5 0.065 -1.6"/>
@@ -815,7 +816,36 @@
   </link>
   <joint name="door_joint" type="fixed">
-    <origin rpy="-1.57 0 0" xyz="0 0 0"/>
+    <origin rpy="3.141592 0 -1.570796" xyz="0 0 0"/>
     <parent link="right_hand_endeffector_link"/>
-    <child link="right_hand_door_link"/>
-  </joint>
+    <child link="right_hand_object_link"/>
+  </joint>
+-->
+<!--
+  <link name="right_hand_object_link">
+    <visual>
+      <origin rpy="0 0 0" xyz="3.1245 -5.3 -1.0819"/>
+      <geometry>
+        <mesh filename="package://move_itomp/meshes/drawer2.dae"/>
+      </geometry>
+      <material name="Blue"/>
+    </visual>
+    <collision>
+      <origin rpy="0 0 0" xyz="3.1245 -5.3 -1.0819"/>
+      <geometry>
+	<mesh filename="package://move_itomp/meshes/drawer2.dae"/>
+      </geometry>
+    </collision>
+  </link>
+  <link name="drawer_dummy"/>
+  <joint name="drawer_joint" type="fixed">
+    <origin rpy="0 -2.468985 0" xyz="0 0 0"/>
+    <parent link="drawer_dummy"/>
+    <child link="right_hand_object_link"/>
+  </joint>
+  <joint name="drawer_joint2" type="fixed">
+    <origin rpy="0 0 0" xyz="0 0 0"/>
+    <parent link="right_hand_endeffector_link"/>
+    <child link="drawer_dummy"/>
+  </joint>
+-->
 </robot>
