Commit message: robot urdf change (add inertia info for all links)

File: human_description/robots/human_cio_rbdl.urdf (robot description, URDF)
Before this commit: robot human_cio, 41 links, 40 joints
Links:
- link head_y_link: mass None -> 0
- link head_z_link: mass None -> 0
- link left_foot_endeffector_link: mass None -> 0
- link left_foot_x_link: mass None -> 0
- link left_foot_y_link: mass None -> 0
- link left_hand_endeffector_link: mass None -> 0
- link left_hand_y_link: mass None -> 0
- link left_hand_z_link: mass None -> 0
- link right_foot_endeffector_link: mass None -> 0
- link right_foot_x_link: mass None -> 0
- link right_foot_y_link: mass None -> 0
- link right_hand_endeffector_link: mass None -> 0
- link right_hand_y_link: mass None -> 0
- link right_hand_z_link: mass None -> 0
- link torso_y_link: mass None -> 0
- link torso_z_link: mass None -> 0
- link upper_left_arm_y_link: mass None -> 0
- link upper_left_arm_z_link: mass None -> 0
- link upper_left_leg_y_link: mass None -> 0
- link upper_left_leg_z_link: mass None -> 0
- link upper_right_arm_y_link: mass None -> 0
- link upper_right_arm_z_link: mass None -> 0
- link upper_right_leg_y_link: mass None -> 0
- link upper_right_leg_z_link: mass None -> 0
