Commit message: itomp_robot_model use RBDL

File: human_description/robots/human_cio.urdf (robot description, URDF)
Before this commit: robot human_cio, 46 links, 45 joints
Joints:
- joint base_revolute_joint_x: child base_revolute_dummy1 -> pelvis_link; parent base_prismatic_dummy3 -> base_revolute_dummy2
- joint base_revolute_joint_z: child pelvis_link -> base_revolute_dummy1; parent base_revolute_dummy2 -> base_prismatic_dummy3

File: human_description/robots/human_cio.urdf.xacro (robot description, xacro)
@@ -105,7 +105,6 @@
     <child link="base_prismatic_dummy3"/>
   </joint>
-  <joint name="base_revolute_joint_x" type="revolute">
-    <axis xyz="1 0 0"/>
-    <limit effort="15" lower="0.0" upper="0.0" velocity="5"/>
+  <joint name="base_revolute_joint_z" type="continuous">
+    <axis xyz="0 0 1"/>
     <origin rpy="0 0 0" xyz="0 0 0"/>
     <parent link="base_prismatic_dummy3"/>
@@ -119,6 +118,7 @@
     <child link="base_revolute_dummy2"/>
   </joint>
-  <joint name="base_revolute_joint_z" type="continuous">
-    <axis xyz="0 0 1"/>
+  <joint name="base_revolute_joint_x" type="revolute">
+    <axis xyz="1 0 0"/>
+    <limit effort="15" lower="0.0" upper="0.0" velocity="5"/>
     <origin rpy="0 0 0" xyz="0 0 0"/>
     <parent link="base_revolute_dummy2"/>

File: human_description/robots/human_cio_rbdl.urdf (robot description, URDF)
Before this commit: robot human_cio, 41 links, 40 joints
Joints:
- joint head_endeffector_joint: type fixed -> continuous
- joint left_foot_endeffector_joint: type fixed -> continuous
- joint left_hand_endeffector_joint: type fixed -> continuous
- joint right_foot_endeffector_joint: type fixed -> continuous
- joint right_hand_endeffector_joint: type fixed -> continuous

Commit message: human model root rotation order : x y z

File: human_description/robots/human_cio.urdf (robot description, URDF)
Before this commit: robot human_cio, 46 links, 45 joints
Joints:
- joint base_revolute_joint_x: child pelvis_link -> base_revolute_dummy1; limit lower=0.0 upper=0.0 effort=15 velocity=5 -> (none); parent base_revolute_dummy2 -> base_prismatic_dummy3; type revolute -> continuous
- joint base_revolute_joint_z: child base_revolute_dummy1 -> pelvis_link; limit (none) -> lower=0.0 upper=0.0 effort=15 velocity=5; parent base_prismatic_dummy3 -> base_revolute_dummy2; type continuous -> revolute

File: human_description/robots/human_cio.urdf.xacro (robot description, xacro)
@@ -105,6 +105,6 @@
     <child link="base_prismatic_dummy3"/>
   </joint>
-  <joint name="base_revolute_joint_z" type="continuous">
-    <axis xyz="0 0 1"/>
+  <joint name="base_revolute_joint_x" type="continuous">
+    <axis xyz="1 0 0"/>
     <origin rpy="0 0 0" xyz="0 0 0"/>
     <parent link="base_prismatic_dummy3"/>
@@ -118,6 +118,6 @@
     <child link="base_revolute_dummy2"/>
   </joint>
-  <joint name="base_revolute_joint_x" type="revolute">
-    <axis xyz="1 0 0"/>
+  <joint name="base_revolute_joint_z" type="revolute">
+    <axis xyz="0 0 1"/>
     <limit effort="15" lower="0.0" upper="0.0" velocity="5"/>
     <origin rpy="0 0 0" xyz="0 0 0"/>

Commit message: modify human model

File: human_description/robots/human_cio.urdf (robot description, URDF)
Before this commit: robot human_cio, 46 links, 45 joints
Joints:
- joint base_revolute_joint_y: limit lower=0.0 upper=0.0 effort=15 velocity=5 -> (none); type revolute -> continuous
- joint base_revolute_joint_z: limit lower=0.0 upper=0.0 effort=15 velocity=5 -> (none); type revolute -> continuous

File: human_description/robots/human_cio.urdf.xacro (robot description, xacro)
@@ -111,14 +111,12 @@
     <child link="base_revolute_dummy1"/>
   </joint>
-  <joint name="base_revolute_joint_y" type="revolute">
-    <axis xyz="0 1 0"/>
-    <limit effort="15" lower="0.0" upper="0.0" velocity="5"/>
+  <joint name="base_revolute_joint_y" type="continuous">
+    <axis xyz="0 1 0"/>
     <origin rpy="0 0 0" xyz="0 0 0"/>
     <parent link="base_revolute_dummy1"/>
     <child link="base_revolute_dummy2"/>
   </joint>
-  <joint name="base_revolute_joint_z" type="revolute">
-    <axis xyz="0 0 1"/>
-    <limit effort="15" lower="0.0" upper="0.0" velocity="5"/>
+  <joint name="base_revolute_joint_z" type="continuous">
+    <axis xyz="0 0 1"/>
     <origin rpy="0 0 0" xyz="0 0 0"/>
     <parent link="base_revolute_dummy2"/>

Commit message: optimization tuning

File: human_description/robots/human_cio.urdf (robot description, URDF)
Before this commit: robot human_cio, 46 links, 45 joints
Links:
- added link left_foot_cp_1_link, mass 0; visual box size=0.001 0.001 0.001
- added link left_foot_cp_2_link, mass 0; visual box size=0.001 0.001 0.001
- added link left_foot_cp_3_link, mass 0; visual box size=0.001 0.001 0.001
- added link left_foot_cp_4_link, mass 0; visual box size=0.001 0.001 0.001
- added link right_foot_cp_1_link, mass 0; visual box size=0.001 0.001 0.001
- added link right_foot_cp_2_link, mass 0; visual box size=0.001 0.001 0.001
- added link right_foot_cp_3_link, mass 0; visual box size=0.001 0.001 0.001
- added link right_foot_cp_4_link, mass 0; visual box size=0.001 0.001 0.001
Joints:
- added joint left_foot_cp_1_joint: type revolute, parent left_foot_z_link, child left_foot_cp_1_link, origin xyz=-0.05 -0.05 -0.1 rpy=0 0 0, axis 0 0 1, limit lower=0 upper=0 effort=15 velocity=5
- added joint left_foot_cp_2_joint: type revolute, parent left_foot_z_link, child left_foot_cp_2_link, origin xyz=0.05 -0.05 -0.1 rpy=0 0 0, axis 0 0 1, limit lower=0 upper=0 effort=15 velocity=5
- added joint left_foot_cp_3_joint: type revolute, parent left_foot_z_link, child left_foot_cp_3_link, origin xyz=0.05 0.2 -0.1 rpy=0 0 0, axis 0 0 1, limit lower=0 upper=0 effort=15 velocity=5
- added joint left_foot_cp_4_joint: type revolute, parent left_foot_z_link, child left_foot_cp_4_link, origin xyz=-0.05 0.2 -0.1 rpy=0 0 0, axis 0 0 1, limit lower=0 upper=0 effort=15 velocity=5
- added joint right_foot_cp_1_joint: type revolute, parent right_foot_z_link, child right_foot_cp_1_link, origin xyz=-0.05 -0.05 -0.1 rpy=0 0 0, axis 0 0 1, limit lower=0 upper=0 effort=15 velocity=5
- added joint right_foot_cp_2_joint: type revolute, parent right_foot_z_link, child right_foot_cp_2_link, origin xyz=0.05 -0.05 -0.1 rpy=0 0 0, axis 0 0 1, limit lower=0 upper=0 effort=15 velocity=5
- added joint right_foot_cp_3_joint: type revolute, parent right_foot_z_link, child right_foot_cp_3_link, origin xyz=0.05 0.2 -0.1 rpy=0 0 0, axis 0 0 1, limit lower=0 upper=0 effort=15 velocity=5
- added joint right_foot_cp_4_joint: type revolute, parent right_foot_z_link, child right_foot_cp_4_link, origin xyz=-0.05 0.2 -0.1 rpy=0 0 0, axis 0 0 1, limit lower=0 upper=0 effort=15 velocity=5

File: human_description/robots/human_cio.urdf.xacro (robot description, xacro)
@@ -847,3 +847,171 @@
   </joint>
 -->
+<link name="left_foot_cp_1_link">
+    <visual>
+      <origin rpy="0 0 0" xyz="0 0 0"/>
+      <geometry>
+        <box size="0.001 0.001 0.001"/>
+      </geometry>
+      <material name="Blue"/>
+    </visual>
+    <inertial>
+      <mass value="0"/>
+      <inertia ixx="1" ixy="0" ixz="0" iyy="1" iyz="0" izz="0"/>
+      <origin xyz="0 0 0"/>
+    </inertial>
+  </link>
+  <link name="left_foot_cp_2_link">
+    <visual>
+      <origin rpy="0 0 0" xyz="0 0 0"/>
+      <geometry>
+        <box size="0.001 0.001 0.001"/>
+      </geometry>
+      <material name="Blue"/>
+    </visual>
+    <inertial>
+      <mass value="0"/>
+      <inertia ixx="1" ixy="0" ixz="0" iyy="1" iyz="0" izz="0"/>
+      <origin xyz="0 0 0"/>
+    </inertial>
+  </link>
+  <link name="left_foot_cp_3_link">
+    <visual>
+      <origin rpy="0 0 0" xyz="0 0 0"/>
+      <geometry>
+        <box size="0.001 0.001 0.001"/>
+      </geometry>
+      <material name="Blue"/>
+    </visual>
+    <inertial>
+      <mass value="0"/>
+      <inertia ixx="1" ixy="0" ixz="0" iyy="1" iyz="0" izz="0"/>
+      <origin xyz="0 0 0"/>
+    </inertial>
+  </link>
+  <link name="left_foot_cp_4_link">
+    <visual>
+      <origin rpy="0 0 0" xyz="0 0 0"/>
+      <geometry>
+        <box size="0.001 0.001 0.001"/>
+      </geometry>
+      <material name="Blue"/>
+    </visual>
+    <inertial>
+      <mass value="0"/>
+      <inertia ixx="1" ixy="0" ixz="0" iyy="1" iyz="0" izz="0"/>
+      <origin xyz="0 0 0"/>
+    </inertial>
+  </link>
+  <joint name="left_foot_cp_1_joint" type="revolute">
+    <axis xyz="0 0 1"/>
+    <limit effort="15" lower="0" upper="0" velocity="5"/>
+    <origin rpy="0 0 0" xyz="-0.05 -0.05 -0.1"/>
+    <parent link="left_foot_z_link"/>
+    <child link="left_foot_cp_1_link"/>
+  </joint>
+  <joint name="left_foot_cp_2_joint" type="revolute">
+    <axis xyz="0 0 1"/>
+    <limit effort="15" lower="0" upper="0" velocity="5"/>
+    <origin rpy="0 0 0" xyz="0.05 -0.05 -0.1"/>
+    <parent link="left_foot_z_link"/>
+    <child link="left_foot_cp_2_link"/>
+  </joint>
+  <joint name="left_foot_cp_3_joint" type="revolute">
+    <axis xyz="0 0 1"/>
+    <limit effort="15" lower="0" upper="0" velocity="5"/>
+    <origin rpy="0 0 0" xyz="0.05 0.2 -0.1"/>
+    <parent link="left_foot_z_link"/>
+    <child link="left_foot_cp_3_link"/>
+  </joint>
+  <joint name="left_foot_cp_4_joint" type="revolute">
+    <axis xyz="0 0 1"/>
+    <limit effort="15" lower="0" upper="0" velocity="5"/>
+    <origin rpy="0 0 0" xyz="-0.05 0.2 -0.1"/>
+    <parent link="left_foot_z_link"/>
+    <child link="left_foot_cp_4_link"/>
+  </joint>
+<link name="right_foot_cp_1_link">
+    <visual>
+      <origin rpy="0 0 0" xyz="0 0 0"/>
+      <geometry>
+        <box size="0.001 0.001 0.001"/>
+      </geometry>
+      <material name="Blue"/>
+    </visual>
+    <inertial>
+      <mass value="0"/>
+      <inertia ixx="1" ixy="0" ixz="0" iyy="1" iyz="0" izz="0"/>
+      <origin xyz="0 0 0"/>
+    </inertial>
+  </link>
+  <link name="right_foot_cp_2_link">
+    <visual>
+      <origin rpy="0 0 0" xyz="0 0 0"/>
+      <geometry>
+        <box size="0.001 0.001 0.001"/>
+      </geometry>
+      <material name="Blue"/>
+    </visual>
+    <inertial>
+      <mass value="0"/>
+      <inertia ixx="1" ixy="0" ixz="0" iyy="1" iyz="0" izz="0"/>
+      <origin xyz="0 0 0"/>
+    </inertial>
+  </link>
+  <link name="right_foot_cp_3_link">
+    <visual>
+      <origin rpy="0 0 0" xyz="0 0 0"/>
+      <geometry>
+        <box size="0.001 0.001 0.001"/>
+      </geometry>
+      <material name="Blue"/>
+    </visual>
+    <inertial>
+      <mass value="0"/>
+      <inertia ixx="1" ixy="0" ixz="0" iyy="1" iyz="0" izz="0"/>
+      <origin xyz="0 0 0"/>
+    </inertial>
+  </link>
+  <link name="right_foot_cp_4_link">
+    <visual>
+      <origin rpy="0 0 0" xyz="0 0 0"/>
+      <geometry>
+        <box size="0.001 0.001 0.001"/>
+      </geometry>
+      <material name="Blue"/>
+    </visual>
+    <inertial>
+      <mass value="0"/>
+      <inertia ixx="1" ixy="0" ixz="0" iyy="1" iyz="0" izz="0"/>
+      <origin xyz="0 0 0"/>
+    </inertial>
+  </link>
+  <joint name="right_foot_cp_1_joint" type="revolute">
+    <axis xyz="0 0 1"/>
+    <limit effort="15" lower="0" upper="0" velocity="5"/>
+    <origin rpy="0 0 0" xyz="-0.05 -0.05 -0.1"/>
+    <parent link="right_foot_z_link"/>
+    <child link="right_foot_cp_1_link"/>
+  </joint>
+  <joint name="right_foot_cp_2_joint" type="revolute">
+    <axis xyz="0 0 1"/>
+    <limit effort="15" lower="0" upper="0" velocity="5"/>
+    <origin rpy="0 0 0" xyz="0.05 -0.05 -0.1"/>
+    <parent link="right_foot_z_link"/>
+    <child link="right_foot_cp_2_link"/>
+  </joint>
+  <joint name="right_foot_cp_3_joint" type="revolute">
+    <axis xyz="0 0 1"/>
+    <limit effort="15" lower="0" upper="0" velocity="5"/>
+    <origin rpy="0 0 0" xyz="0.05 0.2 -0.1"/>
+    <parent link="right_foot_z_link"/>
+    <child link="right_foot_cp_3_link"/>
+  </joint>
+  <joint name="right_foot_cp_4_joint" type="revolute">
+    <axis xyz="0 0 1"/>
+    <limit effort="15" lower="0" upper="0" velocity="5"/>
+    <origin rpy="0 0 0" xyz="-0.05 0.2 -0.1"/>
+    <parent link="right_foot_z_link"/>
+    <child link="right_foot_cp_4_link"/>
+  </joint>
 </robot>

File: human_description/robots/human_cio_rbdl.urdf (robot description, URDF)
Before this commit: robot human_cio, 41 links, 40 joints
Links:
- added link left_foot_cp_1_link, mass 0; visual box size=0.001 0.001 0.001
- added link left_foot_cp_2_link, mass 0; visual box size=0.001 0.001 0.001
- added link left_foot_cp_3_link, mass 0; visual box size=0.001 0.001 0.001
- added link left_foot_cp_4_link, mass 0; visual box size=0.001 0.001 0.001
- added link right_foot_cp_1_link, mass 0; visual box size=0.001 0.001 0.001
- added link right_foot_cp_2_link, mass 0; visual box size=0.001 0.001 0.001
- added link right_foot_cp_3_link, mass 0; visual box size=0.001 0.001 0.001
- added link right_foot_cp_4_link, mass 0; visual box size=0.001 0.001 0.001
Joints:
- added joint left_foot_cp_1_joint: type revolute, parent left_foot_z_link, child left_foot_cp_1_link, origin xyz=-0.05 -0.05 -0.1 rpy=0 0 0, axis 0 0 1, limit lower=0 upper=0 effort=15 velocity=5
- added joint left_foot_cp_2_joint: type revolute, parent left_foot_z_link, child left_foot_cp_2_link, origin xyz=0.05 -0.05 -0.1 rpy=0 0 0, axis 0 0 1, limit lower=0 upper=0 effort=15 velocity=5
- added joint left_foot_cp_3_joint: type revolute, parent left_foot_z_link, child left_foot_cp_3_link, origin xyz=0.05 0.2 -0.1 rpy=0 0 0, axis 0 0 1, limit lower=0 upper=0 effort=15 velocity=5
- added joint left_foot_cp_4_joint: type revolute, parent left_foot_z_link, child left_foot_cp_4_link, origin xyz=-0.05 0.2 -0.1 rpy=0 0 0, axis 0 0 1, limit lower=0 upper=0 effort=15 velocity=5
- added joint right_foot_cp_1_joint: type revolute, parent right_foot_z_link, child right_foot_cp_1_link, origin xyz=-0.05 -0.05 -0.1 rpy=0 0 0, axis 0 0 1, limit lower=0 upper=0 effort=15 velocity=5
- added joint right_foot_cp_2_joint: type revolute, parent right_foot_z_link, child right_foot_cp_2_link, origin xyz=0.05 -0.05 -0.1 rpy=0 0 0, axis 0 0 1, limit lower=0 upper=0 effort=15 velocity=5
- added joint right_foot_cp_3_joint: type revolute, parent right_foot_z_link, child right_foot_cp_3_link, origin xyz=0.05 0.2 -0.1 rpy=0 0 0, axis 0 0 1, limit lower=0 upper=0 effort=15 velocity=5
- added joint right_foot_cp_4_joint: type revolute, parent right_foot_z_link, child right_foot_cp_4_link, origin xyz=-0.05 0.2 -0.1 rpy=0 0 0, axis 0 0 1, limit lower=0 upper=0 effort=15 velocity=5

Commit message: optimization tuning

File: human_description/robots/human_cio.urdf (robot description, URDF)
Before this commit: robot human_cio, 54 links, 53 joints
Joints:
- joint upper_left_leg_x_joint: limit lower=-1.2 upper=1.57 effort=15 velocity=5 -> lower=-0.6 upper=1.0 effort=15 velocity=5; type continuous -> revolute
- joint upper_right_leg_x_joint: limit lower=-1.2 upper=1.57 effort=15 velocity=5 -> lower=-0.6 upper=1.0 effort=15 velocity=5; type continuous -> revolute

File: human_description/robots/human_cio.urdf.xacro (robot description, xacro)
@@ -269,7 +269,7 @@
     <child link="upper_left_leg_y_link"/>
   </joint>
-  <joint name="upper_left_leg_x_joint" type="continuous">
-    <axis xyz="1 0 0"/>
-    <limit effort="15" lower="-1.2" upper="1.57" velocity="5"/>
+  <joint name="upper_left_leg_x_joint" type="revolute">
+    <axis xyz="1 0 0"/>
+    <limit effort="15" lower="-0.6" upper="1.0" velocity="5"/>
     <origin rpy="0 0 0" xyz="0 0 0"/>
     <parent link="upper_left_leg_y_link"/>
@@ -405,7 +405,7 @@
     <child link="upper_right_leg_y_link"/>
   </joint>
-  <joint name="upper_right_leg_x_joint" type="continuous">
-    <axis xyz="1 0 0"/>
-    <limit effort="15" lower="-1.2" upper="1.57" velocity="5"/>
+  <joint name="upper_right_leg_x_joint" type="revolute">
+    <axis xyz="1 0 0"/>
+    <limit effort="15" lower="-0.6" upper="1.0" velocity="5"/>
     <origin rpy="0 0 0" xyz="0 0 0"/>
     <parent link="upper_right_leg_y_link"/>

File: human_description/robots/human_cio_rbdl.urdf (robot description, URDF)
Before this commit: robot human_cio, 49 links, 48 joints
Joints:
- joint upper_left_leg_x_joint: limit lower=-1.2 upper=1.57 effort=15 velocity=5 -> lower=-0.6 upper=1.0 effort=15 velocity=5; type continuous -> revolute
- joint upper_right_leg_x_joint: limit lower=-1.2 upper=1.57 effort=15 velocity=5 -> lower=-0.6 upper=1.0 effort=15 velocity=5; type continuous -> revolute
