Commit message: apartment scene

File: human_description/robots/zoey.urdf.xacro (robot description, xacro)
@@ -4,5 +4,5 @@
        xmlns:interface="http://playerstage.sourceforge.net/gazebo/xmlschema/#interface"
        xmlns:xacro="http://playerstage.sourceforge.net/gazebo/xmlschema/#interface"
-       name="human" >
+       name="zoey" >
   <material name="Blue">
     <color rgba="0.0 0.0 0.8 1.0"/>
@@ -66,5 +66,5 @@
       <origin rpy="0 0 0" xyz="0 0 0"/>
       <geometry>
-        <mesh filename="package://human_description/meshes/zoey/pelvis.dae"/>
+        <mesh filename="package://human_description/meshes/zoey/pelvis.dae" scale="0.00001 0.00001 0.00001"/>
       </geometry>
       <material name="Grey2"/>
@@ -73,5 +73,5 @@
       <origin rpy="0 0 0" xyz="0 0 0"/>
       <geometry>
-        <mesh filename="package://human_description/meshes/zoey/pelvis.dae"/>
+        <mesh filename="package://human_description/meshes/zoey/pelvis.dae" scale="0.00001 0.00001 0.00001"/>
       </geometry>
     </collision>
@@ -111,12 +111,12 @@
       <origin rpy="0 0 0" xyz="0 0 0"/>
       <geometry>
-        <mesh filename="package://human_description/meshes/zoey/torso.dae"/>
-      </geometry>
-      <material name="Blue"/>
-    </visual>
-    <collision>
-      <origin rpy="0 0 0" xyz="0 0 0"/>
-      <geometry>
-        <mesh filename="package://human_description/meshes/zoey/torso.dae"/>
+        <mesh filename="package://human_description/meshes/zoey/torso.dae" scale="0.00001 0.00001 0.00001"/>
+      </geometry>
+      <material name="Blue"/>
+    </visual>
+    <collision>
+      <origin rpy="0 0 0" xyz="0 0 0"/>
+      <geometry>
+        <mesh filename="package://human_description/meshes/zoey/torso.dae" scale="0.00001 0.00001 0.00001"/>
       </geometry>
     </collision>
@@ -150,12 +150,12 @@
       <origin rpy="0 0 0" xyz="0 0 0"/>
       <geometry>
-        <mesh filename="package://human_description/meshes/zoey/head.dae"/>
-      </geometry>
-      <material name="Blue"/>
-    </visual>
-    <collision>
-      <origin rpy="0 0 0" xyz="0 0 0"/>
-      <geometry>
-        <mesh filename="package://human_description/meshes/zoey/head.dae"/>
+        <mesh filename="package://human_description/meshes/zoey/head.dae" scale="100 100 100"/>
+      </geometry>
+      <material name="Blue"/>
+    </visual>
+    <collision>
+      <origin rpy="0 0 0" xyz="0 0 0"/>
+      <geometry>
+        <mesh filename="package://human_description/meshes/zoey/head.dae" scale="100 100 100"/>
       </geometry>
     </collision>
@@ -188,12 +188,12 @@
       <origin rpy="0 0 0" xyz="0 0 0"/>
       <geometry>
-        <mesh filename="package://human_description/meshes/zoey/l_lupperleg.dae"/>
-      </geometry>
-      <material name="Blue"/>
-    </visual>
-    <collision>
-      <origin rpy="0 0 0" xyz="0 0 0"/>
-      <geometry>
-        <mesh filename="package://human_description/meshes/zoey/l_lupperleg.dae"/>
+        <mesh filename="package://human_description/meshes/zoey/l_lupperleg.dae" scale="100 100 100"/>
+      </geometry>
+      <material name="Blue"/>
+    </visual>
+    <collision>
+      <origin rpy="0 0 0" xyz="0 0 0"/>
+      <geometry>
+        <mesh filename="package://human_description/meshes/zoey/l_lupperleg.dae" scale="100 100 100"/>
       </geometry>
     </collision>
@@ -210,12 +210,12 @@
       <origin rpy="0 0 0" xyz="0 0 0"/>
       <geometry>
-        <mesh filename="package://human_description/meshes/zoey/l_lowerleg.dae"/>
-      </geometry>
-      <material name="Blue"/>
-    </visual>
-    <collision>
-      <origin rpy="0 0 0" xyz="0 0 0"/>
-      <geometry>
-        <mesh filename="package://human_description/meshes/zoey/l_lowerleg.dae"/>
+        <mesh filename="package://human_description/meshes/zoey/l_lowerleg.dae" scale="100 100 100"/>
+      </geometry>
+      <material name="Blue"/>
+    </visual>
+    <collision>
+      <origin rpy="0 0 0" xyz="0 0 0"/>
+      <geometry>
+        <mesh filename="package://human_description/meshes/zoey/l_lowerleg.dae" scale="100 100 100"/>
       </geometry>
     </collision>
@@ -248,12 +248,12 @@
       <origin rpy="0 0 0" xyz="0 0 0"/>
       <geometry>
-        <mesh filename="package://human_description/meshes/zoey/l_foot.dae"/>
-      </geometry>
-      <material name="Blue"/>
-    </visual>
-    <collision>
-      <origin rpy="0 0 0" xyz="0 0 0"/>
-      <geometry>
-        <mesh filename="package://human_description/meshes/zoey/l_foot.dae"/>
+        <mesh filename="package://human_description/meshes/zoey/l_foot.dae" scale="100 100 100"/>
+      </geometry>
+      <material name="Blue"/>
+    </visual>
+    <collision>
+      <origin rpy="0 0 0" xyz="0 0 0"/>
+      <geometry>
+        <mesh filename="package://human_description/meshes/zoey/l_foot.dae" scale="100 100 100"/>
       </geometry>
     </collision>
@@ -392,12 +392,12 @@
       <origin rpy="0 0 0" xyz="0 0 0"/>
       <geometry>
-        <mesh filename="package://human_description/meshes/zoey/l_upperarm.dae"/>
-      </geometry>
-      <material name="Blue"/>
-    </visual>
-    <collision>
-      <origin rpy="0 0 0" xyz="0 0 0"/>
-      <geometry>
-        <mesh filename="package://human_description/meshes/zoey/l_upperarm.dae"/>
+        <mesh filename="package://human_description/meshes/zoey/l_upperarm.dae" scale="100 100 100"/>
+      </geometry>
+      <material name="Blue"/>
+    </visual>
+    <collision>
+      <origin rpy="0 0 0" xyz="0 0 0"/>
+      <geometry>
+        <mesh filename="package://human_description/meshes/zoey/l_upperarm.dae" scale="100 100 100"/>
       </geometry>
     </collision>
@@ -414,12 +414,12 @@
       <origin rpy="0 0 0" xyz="0 0 0"/>
       <geometry>
-        <mesh filename="package://human_description/meshes/zoey/l_forearm.dae"/>
-      </geometry>
-      <material name="Blue"/>
-    </visual>
-    <collision>
-      <origin rpy="0 0 0" xyz="0 0 0"/>
-      <geometry>
-        <mesh filename="package://human_description/meshes/zoey/l_forearm.dae"/>
+        <mesh filename="package://human_description/meshes/zoey/l_forearm.dae" scale="100 100 100"/>
+      </geometry>
+      <material name="Blue"/>
+    </visual>
+    <collision>
+      <origin rpy="0 0 0" xyz="0 0 0"/>
+      <geometry>
+        <mesh filename="package://human_description/meshes/zoey/l_forearm.dae" scale="100 100 100"/>
       </geometry>
     </collision>
@@ -452,12 +452,12 @@
       <origin rpy="0 0 0" xyz="0 0 0"/>
       <geometry>
-        <mesh filename="package://human_description/meshes/zoey/l_hand.dae"/>
-      </geometry>
-      <material name="Blue"/>
-    </visual>
-    <collision>
-      <origin rpy="0 0 0" xyz="0 0 0"/>
-      <geometry>
-        <mesh filename="package://human_description/meshes/zoey/l_hand.dae"/>
+        <mesh filename="package://human_description/meshes/zoey/l_hand.dae" scale="100 100 100"/>
+      </geometry>
+      <material name="Blue"/>
+    </visual>
+    <collision>
+      <origin rpy="0 0 0" xyz="0 0 0"/>
+      <geometry>
+        <mesh filename="package://human_description/meshes/zoey/l_hand.dae" scale="100 100 100"/>
       </geometry>
     </collision>
