Commit message: rocketbox moveit config package

File: human_description/robots/rocketbox_male_rbdl.urdf (robot description, URDF)
Before this commit: robot rocketbox_male, 79 links, 78 joints
Links:
- removed link base_prismatic_dummy1
- removed link base_prismatic_dummy2
- removed link base_prismatic_dummy3
- removed link base_revolute_dummy1
- removed link base_revolute_dummy2
Joints:
- removed joint base_prismatic_joint_x
- removed joint base_prismatic_joint_y
- removed joint base_prismatic_joint_z
- removed joint base_revolute_joint_x
- removed joint base_revolute_joint_y
- removed joint base_revolute_joint_z
- added joint root_dummy_joint: type fixed, parent root_link, child pelvis_link

Commit message: model update

File: human_description/robots/rocketbox_male_rbdl.urdf (robot description, URDF)
Before this commit: robot rocketbox_male, 59 links, 58 joints
Joints:
- joint left_hand_endeffector_joint: origin xyz=-0.009816 0.007404 -0.21684 rpy=0 0 0 -> xyz=0.01757 -0.00204 -0.08 rpy=-1.570796 0 1.570796
- joint right_hand_endeffector_joint: origin xyz=-0.000348 0.010884 -0.21684 rpy=0 0 0 -> xyz=-0.01229 -0.007225 -0.07007 rpy=-1.570796 0 -1.570796
