Commit message: replaced dae by obj files

File: human_description/robots/rocketbox_male.urdf (robot description, URDF)
Before this commit: robot rocketbox_male, 60 links, 59 joints
Links:
- link head_x_link: geometry collision mesh filename=package://human_description/meshes/rocket_box/head.obj; visual mesh filename=package://human_description/meshes/rocket_box/head.obj
- link left_foot_x_link: geometry collision mesh filename=package://human_description/meshes/rocket_box/l_foot.obj; visual mesh filename=package://human_description/meshes/rocket_box/l_foot.obj
- link left_hand_x_link: geometry collision mesh filename=package://human_description/meshes/rocket_box/l_hand.obj; visual mesh filename=package://human_description/meshes/rocket_box/l_hand.obj
- link lower_left_arm_link: geometry collision mesh filename=package://human_description/meshes/rocket_box/l_forearm.obj; visual mesh filename=package://human_description/meshes/rocket_box/l_forearm.obj
- link lower_left_leg_link: geometry collision mesh filename=package://human_description/meshes/rocket_box/l_lowerleg.obj; visual mesh filename=package://human_description/meshes/rocket_box/l_lowerleg.obj
- link lower_right_arm_link: geometry collision mesh filename=package://human_description/meshes/rocket_box/r_forearm.obj; visual mesh filename=package://human_description/meshes/rocket_box/r_forearm.obj
- link lower_right_leg_link: geometry collision mesh filename=package://human_description/meshes/rocket_box/r_lowerleg.obj; visual mesh filename=package://human_description/meshes/rocket_box/r_lowerleg.obj
- link right_foot_x_link: geometry collision mesh filename=package://human_description/meshes/rocket_box/r_foot.obj; visual mesh filename=package://human_description/meshes/rocket_box/r_foot.obj
- link right_hand_x_link: geometry collision mesh filename=package://human_description/meshes/rocket_box/r_hand.obj; visual mesh filename=package://human_description/meshes/rocket_box/r_hand.obj
- link torso_x_link: geometry collision mesh filename=package://human_description/meshes/rocket_box/torso.obj; visual mesh filename=package://human_description/meshes/rocket_box/torso.obj
- link upper_left_arm_x_link: geometry collision mesh filename=package://human_description/meshes/rocket_box/l_upperarm.obj; visual mesh filename=package://human_description/meshes/rocket_box/l_upperarm.obj
- link upper_left_leg_x_link: geometry collision mesh filename=package://human_description/meshes/rocket_box/l_lupperleg.o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; visual mesh filename=package://human_description/meshes/rocket_box/l_lupperleg.o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
- link upper_right_arm_x_link: geometry collision mesh filename=package://human_description/meshes/rocket_box/r_upperarm.obj; visual mesh filename=package://human_description/meshes/rocket_box/r_upperarm.obj
- link upper_right_leg_x_link: geometry collision mesh filename=package://human_description/meshes/rocket_box/r_upperleg.obj; visual mesh filename=package://human_description/meshes/rocket_box/r_upperleg.obj

Commit message: rocketbox_male.urdf

File: human_description/robots/rocketbox_male.urdf (robot description, URDF)
Before this commit: robot rocketbox_male, 60 links, 59 joints
Links:
- added link base_prismatic_dummy3; visual box size=0.001 0.001 0.001
- added link base_revolute_dummy1; visual box size=0.001 0.001 0.001
- added link base_revolute_dummy2; visual box size=0.001 0.001 0.001
- added link left_foot_cp_1_link, mass 0; visual box size=0.001 0.001 0.001
- added link left_foot_cp_2_link, mass 0; visual box size=0.001 0.001 0.001
- added link left_foot_cp_3_link, mass 0; visual box size=0.001 0.001 0.001
- added link left_foot_cp_4_link, mass 0; visual box size=0.001 0.001 0.001
- added link left_hand_cp_1_link, mass 0; visual box size=0.001 0.001 0.001
- added link left_hand_cp_2_link, mass 0; visual box size=0.001 0.001 0.001
- added link left_hand_cp_3_link, mass 0; visual box size=0.001 0.001 0.001
- added link left_hand_cp_4_link, mass 0; visual box size=0.001 0.001 0.001
- added link right_foot_cp_1_link, mass 0; visual box size=0.001 0.001 0.001
- added link right_foot_cp_2_link, mass 0; visual box size=0.001 0.001 0.001
- added link right_foot_cp_3_link, mass 0; visual box size=0.001 0.001 0.001
- added link right_foot_cp_4_link, mass 0; visual box size=0.001 0.001 0.001
- added link right_hand_cp_1_link, mass 0; visual box size=0.001 0.001 0.001
- added link right_hand_cp_2_link, mass 0; visual box size=0.001 0.001 0.001
- added link right_hand_cp_3_link, mass 0; visual box size=0.001 0.001 0.001
- added link right_hand_cp_4_link, mass 0; visual box size=0.001 0.001 0.001
- link base_prismatic_dummy1: geometry visual box size=0.001 0.001 0.001
- link base_prismatic_dummy2: geometry visual box size=0.001 0.001 0.001
Joints:
- removed joint base_rotate_joint
- added joint base_prismatic_joint_z: type prismatic, parent base_prismatic_dummy2, child base_prismatic_dummy3, origin xyz=0 0 0 rpy=0 0 0, axis 0 0 1, limit lower=-10.0 upper=10.0 effort=10000 velocity=0.6
- added joint base_revolute_joint_x: type continuous, parent base_prismatic_dummy3, child base_revolute_dummy1, origin xyz=0 0 0 rpy=0 0 0, axis 1 0 0
- added joint base_revolute_joint_y: type continuous, parent base_revolute_dummy1, child base_revolute_dummy2, origin xyz=0 0 0 rpy=0 0 0, axis 0 1 0
- added joint base_revolute_joint_z: type continuous, parent base_revolute_dummy2, child pelvis_link, origin xyz=0 0 0 rpy=0 0 0, axis 0 0 1
- added joint left_foot_cp_1_joint: type revolute, parent left_foot2_x_link, child left_foot_cp_1_link, origin xyz=-0.05 -0.05 -0.1 rpy=0 0 0, axis 0 0 1, limit lower=0 upper=0 effort=15 velocity=5
- added joint left_foot_cp_2_joint: type revolute, parent left_foot2_x_link, child left_foot_cp_2_link, origin xyz=0.05 -0.05 -0.1 rpy=0 0 0, axis 0 0 1, limit lower=0 upper=0 effort=15 velocity=5
- added joint left_foot_cp_3_joint: type revolute, parent left_foot2_x_link, child left_foot_cp_3_link, origin xyz=0.05 0.2 -0.1 rpy=0 0 0, axis 0 0 1, limit lower=0 upper=0 effort=15 velocity=5
- added joint left_foot_cp_4_joint: type revolute, parent left_foot2_x_link, child left_foot_cp_4_link, origin xyz=-0.05 0.2 -0.1 rpy=0 0 0, axis 0 0 1, limit lower=0 upper=0 effort=15 velocity=5
- added joint left_hand_cp_1_joint: type revolute, parent left_hand_x_link, child left_hand_cp_1_link, origin xyz=-0.05 -0.05 -0.1 rpy=0 0 0, axis 0 0 1, limit lower=0 upper=0 effort=15 velocity=5
- added joint left_hand_cp_2_joint: type revolute, parent left_hand_x_link, child left_hand_cp_2_link, origin xyz=0.05 -0.05 -0.1 rpy=0 0 0, axis 0 0 1, limit lower=0 upper=0 effort=15 velocity=5
- added joint left_hand_cp_3_joint: type revolute, parent left_hand_x_link, child left_hand_cp_3_link, origin xyz=0.05 0.2 -0.1 rpy=0 0 0, axis 0 0 1, limit lower=0 upper=0 effort=15 velocity=5
- added joint left_hand_cp_4_joint: type revolute, parent left_hand_x_link, child left_hand_cp_4_link, origin xyz=-0.05 0.2 -0.1 rpy=0 0 0, axis 0 0 1, limit lower=0 upper=0 effort=15 velocity=5
- added joint right_foot_cp_1_joint: type revolute, parent right_foot2_x_link, child right_foot_cp_1_link, origin xyz=-0.05 -0.05 -0.1 rpy=0 0 0, axis 0 0 1, limit lower=0 upper=0 effort=15 velocity=5
- added joint right_foot_cp_2_joint: type revolute, parent right_foot2_x_link, child right_foot_cp_2_link, origin xyz=0.05 -0.05 -0.1 rpy=0 0 0, axis 0 0 1, limit lower=0 upper=0 effort=15 velocity=5
- added joint right_foot_cp_3_joint: type revolute, parent right_foot2_x_link, child right_foot_cp_3_link, origin xyz=0.05 0.2 -0.1 rpy=0 0 0, axis 0 0 1, limit lower=0 upper=0 effort=15 velocity=5
- added joint right_foot_cp_4_joint: type revolute, parent right_foot2_x_link, child right_foot_cp_4_link, origin xyz=-0.05 0.2 -0.1 rpy=0 0 0, axis 0 0 1, limit lower=0 upper=0 effort=15 velocity=5
- added joint right_hand_cp_1_joint: type revolute, parent right_hand_x_link, child right_hand_cp_1_link, origin xyz=-0.05 -0.05 -0.1 rpy=0 0 0, axis 0 0 1, limit lower=0 upper=0 effort=15 velocity=5
- added joint right_hand_cp_2_joint: type revolute, parent right_hand_x_link, child right_hand_cp_2_link, origin xyz=0.05 -0.05 -0.1 rpy=0 0 0, axis 0 0 1, limit lower=0 upper=0 effort=15 velocity=5
- added joint right_hand_cp_3_joint: type revolute, parent right_hand_x_link, child right_hand_cp_3_link, origin xyz=0.05 0.2 -0.1 rpy=0 0 0, axis 0 0 1, limit lower=0 upper=0 effort=15 velocity=5
- added joint right_hand_cp_4_joint: type revolute, parent right_hand_x_link, child right_hand_cp_4_link, origin xyz=-0.05 0.2 -0.1 rpy=0 0 0, axis 0 0 1, limit lower=0 upper=0 effort=15 velocity=5

Commit message: contact points + cleaning extra dofs

File: human_description/robots/rocketbox_male.urdf (robot description, URDF)
Before this commit: robot rocketbox_male, 79 links, 78 joints
Links:
- removed link left_foot2_x_link
- removed link left_foot2_y_link
- removed link left_foot2_z_link
- removed link pelvis1_x_link
- removed link pelvis1_y_link
- removed link pelvis1_z_link
- removed link right_foot2_x_link
- removed link right_foot2_y_link
- removed link right_foot2_z_link
- removed link torso2_x_link
- removed link torso2_y_link
- removed link torso2_z_link
- removed link torso3_x_link
- removed link torso3_y_link
- removed link torso3_z_link
- link head_x_link: mass None -> 16.0164526852
- link left_foot_x_link: mass None -> 2.24629475115
- link left_hand_x_link: mass None -> 0.5669499677
- link lower_left_arm_link: mass None -> 4.1174112191
- link lower_left_leg_link: mass None -> 8.394054321
- link lower_right_arm_link: mass None -> 4.1174112191
- link lower_right_leg_link: mass None -> 8.394054321
- link pelvis_link: mass None -> 24.9873014159
- link right_foot_x_link: mass None -> 2.24629475115
- link right_hand_x_link: mass None -> 0.5669499677
- link torso_x_link: mass None -> 54.1902903318
- link upper_left_arm_x_link: mass None -> 5.0428574576
- link upper_left_leg_x_link: mass None -> 11.28066677275
- link upper_right_arm_x_link: mass None -> 5.0428574576
- link upper_right_leg_x_link: mass None -> 11.28066677275
Joints:
- removed joint left_foot2_x_joint
- removed joint left_foot2_y_joint
- removed joint left_foot2_z_joint
- removed joint pelvis1_x_joint
- removed joint pelvis1_y_joint
- removed joint pelvis1_z_joint
- removed joint right_foot2_x_joint
- removed joint right_foot2_y_joint
- removed joint right_foot2_z_joint
- removed joint torso2_x_joint
- removed joint torso2_y_joint
- removed joint torso2_z_joint
- removed joint torso3_x_joint
- removed joint torso3_y_joint
- removed joint torso3_z_joint
- joint head_z_joint: origin xyz=0 -0.024384 0.079464 rpy=0 0 0 -> xyz=0 -0.020052 .502320 rpy=0 0 0; parent torso3_x_link -> torso_x_link
- joint left_foot_cp_1_joint: origin xyz=-0.05 -0.05 -0.1 rpy=0 0 0 -> xyz=0.08027 0.27372 -0.12195 rpy=0 0 0; parent left_foot2_x_link -> left_foot_x_link
- joint left_foot_cp_2_joint: origin xyz=0.05 -0.05 -0.1 rpy=0 0 0 -> xyz=-0.09166 0.27372 -0.12195 rpy=0 0 0; parent left_foot2_x_link -> left_foot_x_link
- joint left_foot_cp_3_joint: origin xyz=0.05 0.2 -0.1 rpy=0 0 0 -> xyz=-0.09166 -0.07769 -0.12195 rpy=0 0 0; parent left_foot2_x_link -> left_foot_x_link
- joint left_foot_cp_4_joint: origin xyz=-0.05 0.2 -0.1 rpy=0 0 0 -> xyz=0.08027 -0.07769 -0.12195 rpy=0 0 0; parent left_foot2_x_link -> left_foot_x_link
- joint left_foot_endeffector_joint: parent left_foot2_x_link -> left_foot_x_link
- joint left_hand_cp_1_joint: origin xyz=-0.05 -0.05 -0.1 rpy=0 0 0 -> xyz=0.01757 0.0606 -0.22569 rpy=0 0 0
- joint left_hand_cp_2_joint: origin xyz=0.05 -0.05 -0.1 rpy=0 0 0 -> xyz=0.01757 -0.06468 -0.22569 rpy=0 0 0
- joint left_hand_cp_3_joint: origin xyz=0.05 0.2 -0.1 rpy=0 0 0 -> xyz=0.01757 -0.06468 -0.02705 rpy=0 0 0
- joint left_hand_cp_4_joint: origin xyz=-0.05 0.2 -0.1 rpy=0 0 0 -> xyz=0.01757 0.0606 -0.02705 rpy=0 0 0
- joint right_foot_cp_1_joint: origin xyz=-0.05 -0.05 -0.1 rpy=0 0 0 -> xyz=0.10495 0.2684 -0.12195 rpy=0 0 0; parent right_foot2_x_link -> right_foot_x_link
- joint right_foot_cp_2_joint: origin xyz=0.05 -0.05 -0.1 rpy=0 0 0 -> xyz=-0.06698 0.2684 -0.12195 rpy=0 0 0; parent right_foot2_x_link -> right_foot_x_link
- joint right_foot_cp_3_joint: origin xyz=0.05 0.2 -0.1 rpy=0 0 0 -> xyz=-0.06698 -0.08301 -0.12195 rpy=0 0 0; parent right_foot2_x_link -> right_foot_x_link
- joint right_foot_cp_4_joint: origin xyz=-0.05 0.2 -0.1 rpy=0 0 0 -> xyz=0.10495 -0.08301 -0.12195 rpy=0 0 0; parent right_foot2_x_link -> right_foot_x_link
- joint right_foot_endeffector_joint: parent right_foot2_x_link -> right_foot_x_link
- joint right_hand_cp_1_joint: origin xyz=-0.05 -0.05 -0.1 rpy=0 0 0 -> xyz=-0.01229 0.05553 -0.01712 rpy=0 0 0
- joint right_hand_cp_2_joint: origin xyz=0.05 -0.05 -0.1 rpy=0 0 0 -> xyz=-0.01229 -0.06975 -0.01712 rpy=0 0 0
- joint right_hand_cp_3_joint: origin xyz=0.05 0.2 -0.1 rpy=0 0 0 -> xyz=-0.01229 -0.06975 -0.21577 rpy=0 0 0
- joint right_hand_cp_4_joint: origin xyz=-0.05 0.2 -0.1 rpy=0 0 0 -> xyz=-0.01229 0.05553 -0.21577 rpy=0 0 0
- joint torso_z_joint: origin xyz=0 0.008328 0.183624 rpy=0 0 0 -> xyz=0 0.010284 0.327936 rpy=0 0 0; parent pelvis1_x_link -> pelvis_link
- joint upper_left_leg_z_joint: origin xyz=-0.106044 -0.010284 -0.327936 rpy=0 0 0 -> xyz=-0.106044 -0.001956 -0.144312 rpy=0 0 0; parent torso_x_link -> pelvis_link
- joint upper_right_leg_z_joint: origin xyz=0.106044 -0.010284 -0.327924 rpy=0 0 0 -> xyz=0.106044 -0.001956 -0.144300 rpy=0 0 0; parent torso_x_link -> pelvis_link

Commit message: model contact points adjusted

File: human_description/robots/rocketbox_male.urdf (robot description, URDF)
Before this commit: robot rocketbox_male, 64 links, 63 joints
Joints:
- joint base_prismatic_joint_x: limit lower=-5.0 upper=5.0 effort=10000 velocity=0.6 -> lower=-6.0 upper=6.0 effort=10000 velocity=0.6; origin xyz=0 0 1.1713 rpy=0 0 0 -> xyz=0 0 1.218534 rpy=0 0 0
- joint base_prismatic_joint_y: limit lower=-5.0 upper=5.0 effort=10000 velocity=0.6 -> lower=-6.0 upper=6.0 effort=10000 velocity=0.6
- joint left_foot_cp_1_joint: origin xyz=0.08027 0.27372 -0.12195 rpy=0 0 0 -> xyz=0.08027 0.27372 0.0 rpy=0 0 0; parent left_foot_x_link -> left_foot_endeffector_link
- joint left_foot_cp_2_joint: origin xyz=-0.09166 0.27372 -0.12195 rpy=0 0 0 -> xyz=-0.09166 0.27372 0.0 rpy=0 0 0; parent left_foot_x_link -> left_foot_endeffector_link
- joint left_foot_cp_3_joint: origin xyz=-0.09166 -0.07769 -0.12195 rpy=0 0 0 -> xyz=-0.09166 -0.07769 0.0 rpy=0 0 0; parent left_foot_x_link -> left_foot_endeffector_link
- joint left_foot_cp_4_joint: origin xyz=0.08027 -0.07769 -0.12195 rpy=0 0 0 -> xyz=0.08027 -0.07769 0.0 rpy=0 0 0; parent left_foot_x_link -> left_foot_endeffector_link
- joint left_foot_endeffector_joint: limit lower=-0.001 upper=0.001 effort=15 velocity=5 -> lower=0.0 upper=0.0 effort=15 velocity=5; origin xyz=-0.024924 -0.097428 0.001788 rpy=0 0 0 -> xyz=-0.024924 -0.097428 -0.120162 rpy=0 0 0; type fixed -> revolute
- joint right_foot_cp_1_joint: origin xyz=0.10495 0.2684 -0.12195 rpy=0 0 0 -> xyz=0.10495 0.2684 0.0 rpy=0 0 0; parent right_foot_x_link -> right_foot_endeffector_link
- joint right_foot_cp_2_joint: origin xyz=-0.06698 0.2684 -0.12195 rpy=0 0 0 -> xyz=-0.06698 0.2684 0.0 rpy=0 0 0; parent right_foot_x_link -> right_foot_endeffector_link
- joint right_foot_cp_3_joint: origin xyz=-0.06698 -0.08301 -0.12195 rpy=0 0 0 -> xyz=-0.06698 -0.08301 0.0 rpy=0 0 0; parent right_foot_x_link -> right_foot_endeffector_link
- joint right_foot_cp_4_joint: origin xyz=0.10495 -0.08301 -0.12195 rpy=0 0 0 -> xyz=0.10495 -0.08301 0.0 rpy=0 0 0; parent right_foot_x_link -> right_foot_endeffector_link
- joint right_foot_endeffector_joint: limit lower=-0.001 upper=0.001 effort=15 velocity=5 -> lower=0.0 upper=0.0 effort=15 velocity=5; origin xyz=0.024924 -0.097428 0.001776 rpy=0 0 0 -> xyz=0.024924 -0.097428 -0.120162 rpy=0 0 0; type fixed -> revolute

File: human_description/robots/rocketbox_male_rbdl.urdf (robot description, URDF)
Before this commit: robot rocketbox_male, 59 links, 58 joints
Joints:
- joint left_foot_cp_1_joint: origin xyz=0.08027 0.27372 -0.12195 rpy=0 0 0 -> xyz=0.08027 0.27372 0.0 rpy=0 0 0; parent left_foot_x_link -> left_foot_endeffector_link
- joint left_foot_cp_2_joint: origin xyz=-0.09166 0.27372 -0.12195 rpy=0 0 0 -> xyz=-0.09166 0.27372 0.0 rpy=0 0 0; parent left_foot_x_link -> left_foot_endeffector_link
- joint left_foot_cp_3_joint: origin xyz=-0.09166 -0.07769 -0.12195 rpy=0 0 0 -> xyz=-0.09166 -0.07769 0.0 rpy=0 0 0; parent left_foot_x_link -> left_foot_endeffector_link
- joint left_foot_cp_4_joint: origin xyz=0.08027 -0.07769 -0.12195 rpy=0 0 0 -> xyz=0.08027 -0.07769 0.0 rpy=0 0 0; parent left_foot_x_link -> left_foot_endeffector_link
- joint left_foot_endeffector_joint: limit lower=-0.001 upper=0.001 effort=15 velocity=5 -> lower=0.0 upper=0.0 effort=15 velocity=5; origin xyz=-0.024924 -0.097428 0.001788 rpy=0 0 0 -> xyz=-0.024924 -0.097428 -0.120162 rpy=0 0 0; type fixed -> revolute
- joint right_foot_cp_1_joint: origin xyz=0.10495 0.2684 -0.12195 rpy=0 0 0 -> xyz=0.10495 0.2684 0.0 rpy=0 0 0; parent right_foot_x_link -> right_foot_endeffector_link
- joint right_foot_cp_2_joint: origin xyz=-0.06698 0.2684 -0.12195 rpy=0 0 0 -> xyz=-0.06698 0.2684 0.0 rpy=0 0 0; parent right_foot_x_link -> right_foot_endeffector_link
- joint right_foot_cp_3_joint: origin xyz=-0.06698 -0.08301 -0.12195 rpy=0 0 0 -> xyz=-0.06698 -0.08301 0.0 rpy=0 0 0; parent right_foot_x_link -> right_foot_endeffector_link
- joint right_foot_cp_4_joint: origin xyz=0.10495 -0.08301 -0.12195 rpy=0 0 0 -> xyz=0.10495 -0.08301 0.0 rpy=0 0 0; parent right_foot_x_link -> right_foot_endeffector_link
- joint right_foot_endeffector_joint: limit lower=-0.001 upper=0.001 effort=15 velocity=5 -> lower=0.0 upper=0.0 effort=15 velocity=5; origin xyz=0.024924 -0.097428 0.001776 rpy=0 0 0 -> xyz=0.024924 -0.097428 -0.120162 rpy=0 0 0; type fixed -> revolute

Commit message: read contact points from params_zombie.yaml

File: human_description/robots/rocketbox_male.urdf (robot description, URDF)
Before this commit: robot rocketbox_male, 64 links, 63 joints
Joints:
- joint left_foot_endeffector_joint: origin xyz=-0.024924 -0.097428 -0.120162 rpy=0 0 0 -> xyz=0 0 -0.120162 rpy=0 0 0
- joint right_foot_endeffector_joint: origin xyz=0.024924 -0.097428 -0.120162 rpy=0 0 0 -> xyz=0 0 -0.120162 rpy=0 0 0

File: human_description/robots/rocketbox_male_rbdl.urdf (robot description, URDF)
Before this commit: robot rocketbox_male, 59 links, 58 joints
Joints:
- joint left_foot_endeffector_joint: origin xyz=-0.024924 -0.097428 -0.120162 rpy=0 0 0 -> xyz=0 0 -0.120162 rpy=0 0 0
- joint right_foot_endeffector_joint: origin xyz=0.024924 -0.097428 -0.120162 rpy=0 0 0 -> xyz=0 0 -0.120162 rpy=0 0 0

Commit message: modify model hand contact points

File: human_description/robots/rocketbox_male.urdf (robot description, URDF)
Before this commit: robot rocketbox_male, 64 links, 63 joints
Joints:
- joint left_hand_cp_1_joint: origin xyz=0.01757 0.0606 -0.22569 rpy=0 0 0 -> xyz=0.06264 0.14569 0 rpy=0 0 0; parent left_hand_x_link -> left_hand_endeffector_link
- joint left_hand_cp_2_joint: origin xyz=0.01757 -0.06468 -0.22569 rpy=0 0 0 -> xyz=-0.06264 0.14569 0 rpy=0 0 0; parent left_hand_x_link -> left_hand_endeffector_link
- joint left_hand_cp_3_joint: origin xyz=0.01757 -0.06468 -0.02705 rpy=0 0 0 -> xyz=-0.06264 -0.05295 0 rpy=0 0 0; parent left_hand_x_link -> left_hand_endeffector_link
- joint left_hand_cp_4_joint: origin xyz=0.01757 0.0606 -0.02705 rpy=0 0 0 -> xyz=0.06264 -0.05295 0 rpy=0 0 0; parent left_hand_x_link -> left_hand_endeffector_link
- joint left_hand_endeffector_joint: origin xyz=-0.009816 0.007404 -0.21684 rpy=0 0 0 -> xyz=0.01757 -0.00204 -0.08 rpy=-1.570796 0 1.570796
- joint right_hand_cp_1_joint: origin xyz=-0.01229 0.05553 -0.01712 rpy=0 0 0 -> xyz=-0.06264 -0.05295 0 rpy=0 0 0; parent right_hand_x_link -> right_hand_endeffector_link
- joint right_hand_cp_2_joint: origin xyz=-0.01229 -0.06975 -0.01712 rpy=0 0 0 -> xyz=0.06264 -0.05295 0 rpy=0 0 0; parent right_hand_x_link -> right_hand_endeffector_link
- joint right_hand_cp_3_joint: origin xyz=-0.01229 -0.06975 -0.21577 rpy=0 0 0 -> xyz=0.06264 0.1457 0 rpy=0 0 0; parent right_hand_x_link -> right_hand_endeffector_link
- joint right_hand_cp_4_joint: origin xyz=-0.01229 0.05553 -0.21577 rpy=0 0 0 -> xyz=-0.06264 0.1457 0 rpy=0 0 0; parent right_hand_x_link -> right_hand_endeffector_link
- joint right_hand_endeffector_joint: origin xyz=-0.000348 0.010884 -0.21684 rpy=0 0 0 -> xyz=-0.01229 -0.007225 -0.07007 rpy=-1.570796 0 -1.570796

File: human_description/robots/rocketbox_male_rbdl.urdf (robot description, URDF)
Before this commit: robot rocketbox_male, 59 links, 58 joints
Joints:
- joint left_hand_cp_1_joint: origin xyz=0.01757 0.0606 -0.22569 rpy=0 0 0 -> xyz=0.06264 0.14569 0 rpy=0 0 0; parent left_hand_x_link -> left_hand_endeffector_link
- joint left_hand_cp_2_joint: origin xyz=0.01757 -0.06468 -0.22569 rpy=0 0 0 -> xyz=-0.06264 0.14569 0 rpy=0 0 0; parent left_hand_x_link -> left_hand_endeffector_link
- joint left_hand_cp_3_joint: origin xyz=0.01757 -0.06468 -0.02705 rpy=0 0 0 -> xyz=-0.06264 -0.05295 0 rpy=0 0 0; parent left_hand_x_link -> left_hand_endeffector_link
- joint left_hand_cp_4_joint: origin xyz=0.01757 0.0606 -0.02705 rpy=0 0 0 -> xyz=0.06264 -0.05295 0 rpy=0 0 0; parent left_hand_x_link -> left_hand_endeffector_link
- joint right_hand_cp_1_joint: origin xyz=-0.01229 0.05553 -0.01712 rpy=0 0 0 -> xyz=-0.06264 -0.05295 0 rpy=0 0 0; parent right_hand_x_link -> right_hand_endeffector_link
- joint right_hand_cp_2_joint: origin xyz=-0.01229 -0.06975 -0.01712 rpy=0 0 0 -> xyz=0.06264 -0.05295 0 rpy=0 0 0; parent right_hand_x_link -> right_hand_endeffector_link
- joint right_hand_cp_3_joint: origin xyz=-0.01229 -0.06975 -0.21577 rpy=0 0 0 -> xyz=0.06264 0.1457 0 rpy=0 0 0; parent right_hand_x_link -> right_hand_endeffector_link
- joint right_hand_cp_4_joint: origin xyz=-0.01229 0.05553 -0.21577 rpy=0 0 0 -> xyz=-0.06264 0.1457 0 rpy=0 0 0; parent right_hand_x_link -> right_hand_endeffector_link
