Commit message: remove joint limits

File: human_description/robots/rocketbox_male.urdf (robot description, URDF)
Before this commit: robot rocketbox_male, 64 links, 63 joints
Joints:
- joint base_prismatic_joint_x: limit lower=-6.0 upper=6.0 effort=10000 velocity=0.6 -> lower=-60.0 upper=60.0 effort=10000 velocity=0.6
- joint base_prismatic_joint_y: limit lower=-6.0 upper=6.0 effort=10000 velocity=0.6 -> lower=-60.0 upper=60.0 effort=10000 velocity=0.6
- joint base_prismatic_joint_z: limit lower=-10.0 upper=10.0 effort=10000 velocity=0.6 -> lower=-100.0 upper=100.0 effort=10000 velocity=0.6
- joint head_x_joint: type revolute -> continuous
- joint head_y_joint: type revolute -> continuous
- joint head_z_joint: type revolute -> continuous
- joint left_foot_x_joint: type revolute -> continuous
- joint left_foot_y_joint: type revolute -> continuous
- joint left_foot_z_joint: type revolute -> continuous
- joint left_hand_x_joint: type revolute -> continuous
- joint left_hand_y_joint: type revolute -> continuous
- joint left_hand_z_joint: type revolute -> continuous
- joint lower_left_arm_joint: type revolute -> continuous
- joint lower_left_leg_joint: type revolute -> continuous
- joint lower_right_arm_joint: type revolute -> continuous
- joint lower_right_leg_joint: type revolute -> continuous
- joint right_foot_x_joint: type revolute -> continuous
- joint right_foot_y_joint: type revolute -> continuous
- joint right_foot_z_joint: type revolute -> continuous
- joint right_hand_x_joint: type revolute -> continuous
- joint right_hand_y_joint: type revolute -> continuous
- joint right_hand_z_joint: type revolute -> continuous
- joint torso_x_joint: type revolute -> continuous
- joint torso_y_joint: type revolute -> continuous
- joint torso_z_joint: type revolute -> continuous
- joint upper_left_arm_x_joint: type revolute -> continuous
- joint upper_left_arm_y_joint: type revolute -> continuous
- joint upper_left_arm_z_joint: type revolute -> continuous
- joint upper_left_leg_x_joint: type revolute -> continuous
- joint upper_left_leg_y_joint: type revolute -> continuous
- joint upper_left_leg_z_joint: type revolute -> continuous
- joint upper_left_specula_joint: type revolute -> continuous
- joint upper_right_arm_x_joint: type revolute -> continuous
- joint upper_right_arm_y_joint: type revolute -> continuous
- joint upper_right_arm_z_joint: type revolute -> continuous
- joint upper_right_leg_x_joint: type revolute -> continuous
- joint upper_right_leg_y_joint: type revolute -> continuous
- joint upper_right_leg_z_joint: type revolute -> continuous
- joint upper_right_specula_joint: type revolute -> continuous

File: human_description/robots/rocketbox_male_rbdl.urdf (robot description, URDF)
Before this commit: robot rocketbox_male, 59 links, 58 joints
Joints:
- joint head_x_joint: type revolute -> continuous
- joint head_y_joint: type revolute -> continuous
- joint head_z_joint: type revolute -> continuous
- joint left_foot_x_joint: type revolute -> continuous
- joint left_foot_y_joint: type revolute -> continuous
- joint left_foot_z_joint: type revolute -> continuous
- joint left_hand_x_joint: type revolute -> continuous
- joint left_hand_y_joint: type revolute -> continuous
- joint left_hand_z_joint: type revolute -> continuous
- joint lower_left_arm_joint: type revolute -> continuous
- joint lower_left_leg_joint: type revolute -> continuous
- joint lower_right_arm_joint: type revolute -> continuous
- joint lower_right_leg_joint: type revolute -> continuous
- joint right_foot_x_joint: type revolute -> continuous
- joint right_foot_y_joint: type revolute -> continuous
- joint right_foot_z_joint: type revolute -> continuous
- joint right_hand_x_joint: type revolute -> continuous
- joint right_hand_y_joint: type revolute -> continuous
- joint right_hand_z_joint: type revolute -> continuous
- joint torso_x_joint: type revolute -> continuous
- joint torso_y_joint: type revolute -> continuous
- joint torso_z_joint: type revolute -> continuous
- joint upper_left_arm_x_joint: type revolute -> continuous
- joint upper_left_arm_y_joint: type revolute -> continuous
- joint upper_left_arm_z_joint: type revolute -> continuous
- joint upper_left_leg_x_joint: type revolute -> continuous
- joint upper_left_leg_y_joint: type revolute -> continuous
- joint upper_left_leg_z_joint: type revolute -> continuous
- joint upper_left_specula_joint: type revolute -> continuous
- joint upper_right_arm_x_joint: type revolute -> continuous
- joint upper_right_arm_y_joint: type revolute -> continuous
- joint upper_right_arm_z_joint: type revolute -> continuous
- joint upper_right_leg_x_joint: type revolute -> continuous
- joint upper_right_leg_y_joint: type revolute -> continuous
- joint upper_right_leg_z_joint: type revolute -> continuous
- joint upper_right_specula_joint: type revolute -> continuous

Commit message: remove geometries of vitrual links

File: human_description/robots/rocketbox_male.urdf (robot description, URDF)
Before this commit: robot rocketbox_male, 64 links, 63 joints
Links:
- link base_prismatic_dummy1: geometry 
- link base_prismatic_dummy2: geometry 
- link base_prismatic_dummy3: geometry 
- link base_revolute_dummy1: geometry 
- link base_revolute_dummy2: geometry 
- link head_endeffector_link: geometry 
- link left_foot_cp_1_link: mass 0 -> None; geometry 
- link left_foot_cp_2_link: mass 0 -> None; geometry 
- link left_foot_cp_3_link: mass 0 -> None; geometry 
- link left_foot_cp_4_link: mass 0 -> None; geometry 
- link left_foot_endeffector_link: geometry 
- link left_hand_cp_1_link: mass 0 -> None; geometry 
- link left_hand_cp_2_link: mass 0 -> None; geometry 
- link left_hand_cp_3_link: mass 0 -> None; geometry 
- link left_hand_cp_4_link: mass 0 -> None; geometry 
- link left_hand_endeffector_link: geometry 
- link right_foot_cp_1_link: mass 0 -> None; geometry 
- link right_foot_cp_2_link: mass 0 -> None; geometry 
- link right_foot_cp_3_link: mass 0 -> None; geometry 
- link right_foot_cp_4_link: mass 0 -> None; geometry 
- link right_foot_endeffector_link: geometry 
- link right_hand_cp_1_link: mass 0 -> None; geometry 
- link right_hand_cp_2_link: mass 0 -> None; geometry 
- link right_hand_cp_3_link: mass 0 -> None; geometry 
- link right_hand_cp_4_link: mass 0 -> None; geometry 
- link right_hand_endeffector_link: geometry 

File: human_description/robots/rocketbox_male_rbdl.urdf (robot description, URDF)
Before this commit: robot rocketbox_male, 59 links, 58 joints
Links:
- link head_endeffector_link: geometry 
- link left_foot_cp_1_link: mass 0 -> None; geometry 
- link left_foot_cp_2_link: mass 0 -> None; geometry 
- link left_foot_cp_3_link: mass 0 -> None; geometry 
- link left_foot_cp_4_link: mass 0 -> None; geometry 
- link left_foot_endeffector_link: geometry 
- link left_hand_cp_1_link: mass 0 -> None; geometry 
- link left_hand_cp_2_link: mass 0 -> None; geometry 
- link left_hand_cp_3_link: mass 0 -> None; geometry 
- link left_hand_cp_4_link: mass 0 -> None; geometry 
- link left_hand_endeffector_link: geometry 
- link right_foot_cp_1_link: mass 0 -> None; geometry 
- link right_foot_cp_2_link: mass 0 -> None; geometry 
- link right_foot_cp_3_link: mass 0 -> None; geometry 
- link right_foot_cp_4_link: mass 0 -> None; geometry 
- link right_foot_endeffector_link: geometry 
- link right_hand_cp_1_link: mass 0 -> None; geometry 
- link right_hand_cp_2_link: mass 0 -> None; geometry 
- link right_hand_cp_3_link: mass 0 -> None; geometry 
- link right_hand_cp_4_link: mass 0 -> None; geometry 
- link right_hand_endeffector_link: geometry 

Commit message: adjust model urdf

File: human_description/robots/rocketbox_male.urdf (robot description, URDF)
Before this commit: robot rocketbox_male, 64 links, 63 joints
Links:
- link head_x_link: mass 16.0164526852 -> 16.0
- link left_foot_x_link: mass 2.24629475115 -> 2.25
- link left_hand_x_link: mass 0.5669499677 -> 0.57
- link lower_left_arm_link: mass 4.1174112191 -> 4.12
- link lower_left_leg_link: mass 8.394054321 -> 8.39
- link lower_right_arm_link: mass 4.1174112191 -> 4.12
- link lower_right_leg_link: mass 8.394054321 -> 8.39
- link pelvis_link: mass 24.9873014159 -> 25.0
- link right_foot_x_link: mass 2.24629475115 -> 2.25
- link right_hand_x_link: mass 0.5669499677 -> 0.57
- link torso_x_link: mass 54.1902903318 -> 54.20
- link upper_left_arm_x_link: mass 5.0428574576 -> 5.04
- link upper_left_leg_x_link: mass 11.28066677275 -> 11.28
- link upper_right_arm_x_link: mass 5.0428574576 -> 5.04
- link upper_right_leg_x_link: mass 11.28066677275 -> 11.28
Joints:
- joint base_prismatic_joint_x: origin xyz=0 0 1.218534 rpy=0 0 0 -> xyz=0 0 1.21 rpy=0 0 0
- joint head_endeffector_joint: origin xyz=0 -0.03768 0.246336 rpy=0 0 0 -> xyz=0 -0.04 0.25 rpy=0 0 0
- joint head_z_joint: origin xyz=0 -0.020052 .502320 rpy=0 0 0 -> xyz=0 0 0.5 rpy=0 0 0
- joint left_foot_cp_1_joint: origin xyz=0.08027 0.27372 0.0 rpy=0 0 0 -> xyz=0.08 0.27 0.0 rpy=0 0 0
- joint left_foot_cp_2_joint: origin xyz=-0.09166 0.27372 0.0 rpy=0 0 0 -> xyz=-0.08 0.27 0.0 rpy=0 0 0
- joint left_foot_cp_3_joint: origin xyz=-0.09166 -0.07769 0.0 rpy=0 0 0 -> xyz=-0.08 -0.08 0.0 rpy=0 0 0
- joint left_foot_cp_4_joint: origin xyz=0.08027 -0.07769 0.0 rpy=0 0 0 -> xyz=0.08 -0.08 0.0 rpy=0 0 0
- joint left_foot_endeffector_joint: origin xyz=0 0 -0.120162 rpy=0 0 0 -> xyz=0 0 -0.12 rpy=0 0 0
- joint left_foot_z_joint: origin xyz=-0.008988 0.036996 -0.474504 rpy=0 0 0 -> xyz=-0.01 0.04 -0.47 rpy=0 0 0
- joint left_hand_cp_1_joint: origin xyz=0.06264 0.14569 0 rpy=0 0 0 -> xyz=0.06 0.14 0 rpy=0 0 0
- joint left_hand_cp_2_joint: origin xyz=-0.06264 0.14569 0 rpy=0 0 0 -> xyz=-0.06 0.14 0 rpy=0 0 0
- joint left_hand_cp_3_joint: origin xyz=-0.06264 -0.05295 0 rpy=0 0 0 -> xyz=-0.06 -0.05 0 rpy=0 0 0
- joint left_hand_cp_4_joint: origin xyz=0.06264 -0.05295 0 rpy=0 0 0 -> xyz=0.06 -0.05 0 rpy=0 0 0
- joint left_hand_endeffector_joint: origin xyz=0.01757 -0.00204 -0.08 rpy=-1.570796 0 1.570796 -> xyz=0.015 -0.01 -0.08 rpy=-1.570796 0 1.570796
- joint left_hand_z_joint: origin xyz=-0.001728 -0.004992 -0.325056 rpy=0 0 0 -> xyz=0.0 0.0 -0.32 rpy=0 0 0
- joint lower_left_arm_joint: origin xyz=-0.001464 -0.00114 -0.34296 rpy=0 0 0 -> xyz=0.0 0.0 -0.34 rpy=0 0 0
- joint lower_left_leg_joint: origin xyz=-0.025332 -0.01956 -0.477768 rpy=0 0 0 -> xyz=-0.03 -0.02 -0.48 rpy=0 0 0
- joint lower_right_arm_joint: origin xyz=-0.005592 -0.007404 -0.342828 rpy=0 0 0 -> xyz=0.0 0.0 -0.34 rpy=0 0 0
- joint lower_right_leg_joint: origin xyz=0.025332 -0.01956 -0.47778 rpy=0 0 0 -> xyz=0.03 -0.02 -0.48 rpy=0 0 0
- joint right_foot_cp_1_joint: origin xyz=0.10495 0.2684 0.0 rpy=0 0 0 -> xyz=0.08 0.27 0.0 rpy=0 0 0
- joint right_foot_cp_2_joint: origin xyz=-0.06698 0.2684 0.0 rpy=0 0 0 -> xyz=-0.08 0.27 0.0 rpy=0 0 0
- joint right_foot_cp_3_joint: origin xyz=-0.06698 -0.08301 0.0 rpy=0 0 0 -> xyz=-0.08 -0.08 0.0 rpy=0 0 0
- joint right_foot_cp_4_joint: origin xyz=0.10495 -0.08301 0.0 rpy=0 0 0 -> xyz=0.08 -0.08 0.0 rpy=0 0 0
- joint right_foot_endeffector_joint: origin xyz=0 0 -0.120162 rpy=0 0 0 -> xyz=0 0 -0.12 rpy=0 0 0
- joint right_foot_z_joint: origin xyz=0.008988 0.036996 -0.474504 rpy=0 0 0 -> xyz=0.01 0.04 -0.47 rpy=0 0 0
- joint right_hand_cp_1_joint: origin xyz=-0.06264 -0.05295 0 rpy=0 0 0 -> xyz=-0.06 -0.05 0 rpy=0 0 0
- joint right_hand_cp_2_joint: origin xyz=0.06264 -0.05295 0 rpy=0 0 0 -> xyz=0.06 -0.05 0 rpy=0 0 0
- joint right_hand_cp_3_joint: origin xyz=0.06264 0.1457 0 rpy=0 0 0 -> xyz=0.06 0.14 0 rpy=0 0 0
- joint right_hand_cp_4_joint: origin xyz=-0.06264 0.1457 0 rpy=0 0 0 -> xyz=-0.06 0.14 0 rpy=0 0 0
- joint right_hand_endeffector_joint: origin xyz=-0.01229 -0.007225 -0.07007 rpy=-1.570796 0 -1.570796 -> xyz=-0.015 -0.01 -0.08 rpy=-1.570796 0 -1.570796
- joint right_hand_z_joint: origin xyz=-0.004728 -0.003084 -0.325056 rpy=0 0 0 -> xyz=0.0 0.0 -0.32 rpy=0 0 0
- joint torso_z_joint: origin xyz=0 0.010284 0.327936 rpy=0 0 0 -> xyz=0 0.0 0.33 rpy=0 0 0
- joint upper_left_arm_z_joint: origin xyz=-0.169296 0 0 rpy=0 0 0 -> xyz=-0.17 0 0 rpy=0 0 0
- joint upper_left_leg_z_joint: origin xyz=-0.106044 -0.001956 -0.144312 rpy=0 0 0 -> xyz=-0.10 0.0 -0.14 rpy=0 0 0
- joint upper_left_specula_joint: origin xyz=-0.0873828 0.0381 -0.153156 rpy=0 0 0 -> xyz=-0.09 0.04 0.35 rpy=0 0 0; parent head_x_link -> torso_x_link
- joint upper_right_arm_z_joint: origin xyz=0.16926 0.003768 -0.0003 rpy=0 0 0 -> xyz=0.17 0.0 0.0 rpy=0 0 0
- joint upper_right_leg_z_joint: origin xyz=0.106044 -0.001956 -0.144300 rpy=0 0 0 -> xyz=0.10 0.0 -0.14 rpy=0 0 0
- joint upper_right_specula_joint: axis 1 0 0 -> 0 0 1; origin xyz=0.0873852 0.0381 -0.153312 rpy=0 0 0 -> xyz=0.09 0.04 0.35 rpy=0 0 0; parent head_x_link -> torso_x_link

Commit message: modify model to avoid initial collision between torso and left arm

File: human_description/robots/rocketbox_male.urdf (robot description, URDF)
Before this commit: robot rocketbox_male, 64 links, 63 joints
Joints:
- joint upper_left_specula_joint: origin xyz=-0.09 0.04 0.35 rpy=0 0 0 -> xyz=-0.12 0.04 0.35 rpy=0 0 0
- joint upper_right_specula_joint: origin xyz=0.09 0.04 0.35 rpy=0 0 0 -> xyz=0.12 0.04 0.35 rpy=0 0 0

Commit message: set model weight to 60

File: human_description/robots/rocketbox_male.urdf (robot description, URDF)
Before this commit: robot rocketbox_male, 64 links, 63 joints
Links:
- link head_x_link: mass 16.0 -> 4.0
- link left_foot_x_link: mass 2.25 -> 1.0
- link left_hand_x_link: mass 0.57 -> 0.25
- link lower_left_arm_link: mass 4.12 -> 1.5
- link lower_left_leg_link: mass 8.39 -> 3.0
- link lower_right_arm_link: mass 4.12 -> 1.5
- link lower_right_leg_link: mass 8.39 -> 3.0
- link pelvis_link: mass 25.0 -> 11.5
- link right_foot_x_link: mass 2.25 -> 1.0
- link right_hand_x_link: mass 0.57 -> 0.25
- link torso_x_link: mass 54.20 -> 20.0
- link upper_left_arm_x_link: mass 5.04 -> 2.0
- link upper_left_leg_x_link: mass 11.28 -> 4.5
- link upper_right_arm_x_link: mass 5.04 -> 2.0
- link upper_right_leg_x_link: mass 11.28 -> 4.5

Commit message: make the right hand potential contact points have the same order with the left hand

File: human_description/robots/rocketbox_male.urdf (robot description, URDF)
Before this commit: robot rocketbox_male, 64 links, 63 joints
Joints:
- joint right_hand_cp_1_joint: origin xyz=-0.06 -0.05 0 rpy=0 0 0 -> xyz=0.06 0.14 0 rpy=0 0 0
- joint right_hand_cp_2_joint: origin xyz=0.06 -0.05 0 rpy=0 0 0 -> xyz=-0.06 0.14 0 rpy=0 0 0
- joint right_hand_cp_3_joint: origin xyz=0.06 0.14 0 rpy=0 0 0 -> xyz=-0.06 -0.05 0 rpy=0 0 0
- joint right_hand_cp_4_joint: origin xyz=-0.06 0.14 0 rpy=0 0 0 -> xyz=0.06 -0.05 0 rpy=0 0 0
