Commit message: lbr3 model update

File: lbr3_model/lbr_gripper_pinch.urdf (robot description, URDF)
Before this commit: robot lbr3, 19 links, 18 joints
Links:
- added link link_kinect; visual box size=0.6 2.8 .4
Joints:
- added joint kinect_depth_joint: type fixed, parent segment_0, child link_kinect, origin xyz=5.15 9.6 14.55 rpy=0 0.87 -1.57

Commit message: adjust scale

File: lbr3_model/lbr_gripper_pinch.urdf (robot description, URDF)
Before this commit: robot lbr3, 20 links, 19 joints
Links:
- link link_kinect: geometry visual box size=0.06 0.28 .04
- link segment_0: geometry collision mesh filename=package://lbr3_model/cad/segment_0_collision.dae scale=0.001 0.001 0.001; visual mesh filename=package://lbr3_model/cad/segment_0.dae scale=0.001 0.001 0.001
- link segment_1: geometry collision mesh filename=package://lbr3_model/cad/segment_1_collision.dae scale=0.001 0.001 0.001; visual mesh filename=package://lbr3_model/cad/segment_1.dae scale=0.001 0.001 0.001
- link segment_2: geometry collision mesh filename=package://lbr3_model/cad/segment_2_collision.dae scale=0.001 0.001 0.001; visual mesh filename=package://lbr3_model/cad/segment_2.dae scale=0.001 0.001 0.001
- link segment_3: geometry collision mesh filename=package://lbr3_model/cad/segment_3_collision.dae scale=0.001 0.001 0.001; visual mesh filename=package://lbr3_model/cad/segment_3.dae scale=0.001 0.001 0.001
- link segment_4: geometry collision mesh filename=package://lbr3_model/cad/segment_4_collision.dae scale=0.001 0.001 0.001; visual mesh filename=package://lbr3_model/cad/segment_4.dae scale=0.001 0.001 0.001
- link segment_5: geometry collision mesh filename=package://lbr3_model/cad/segment_5_collision.dae scale=0.001 0.001 0.001; visual mesh filename=package://lbr3_model/cad/segment_5.dae scale=0.001 0.001 0.001
- link segment_6: geometry collision mesh filename=package://lbr3_model/cad/segment_6_collision.dae scale=0.001 0.001 0.001; visual mesh filename=package://lbr3_model/cad/segment_6.dae scale=0.001 0.001 0.001
- link segment_7: geometry collision mesh filename=package://lbr3_model/cad/segment_7_collision.dae scale=0.001 0.001 0.001; visual mesh filename=package://lbr3_model/cad/segment_7.dae scale=0.001 0.001 0.001
- link tool: geometry collision mesh filename=package://kuka_description/cad/tool.dae scale=0.001 0.001 0.001; visual mesh filename=package://kuka_description/cad/tool.dae scale=0.001 0.001 0.001
Joints:
- joint joint_0: origin xyz=0 0 1.105 -> xyz=0 0 .1105
- joint joint_1: origin xyz=0 0 2 -> xyz=0 0 .2
- joint joint_2: origin xyz=0 0 2 -> xyz=0 0 .2
- joint joint_3: origin xyz=0 0 2 -> xyz=0 0 .2
- joint joint_4: origin xyz=0 0 2 -> xyz=0 0 .2
- joint joint_5: origin xyz=0 0 1.885 -> xyz=0 0 .1885
- joint joint_6: origin xyz=0 0 .795 -> xyz=0 0 .0795
- joint joint_goal_2: origin xyz=2.0 1.0 12.0 rpy=-1.570796 0 1.570796 -> xyz=.20 .10 1.20 rpy=-1.570796 0 1.570796
- joint joint_goal_3: origin xyz=2.0 1.5 12.0 rpy=-1.570796 0 1.570796 -> xyz=.20 .15 1.20 rpy=-1.570796 0 1.570796
- joint joint_goal_4: origin xyz=2.0 2.0 8.5 rpy=-1.570796 0 3.141592 -> xyz=.20 .20 .85 rpy=-1.570796 0 3.141592
- joint joint_goal_5: origin xyz=1.5 2.0 8.5 rpy=-1.570796 0 3.141592 -> xyz=.15 .20 .85 rpy=-1.570796 0 3.141592
- joint joint_goal_6: origin xyz=1.0 2.0 8.5 rpy=-1.570796 0 3.141592 -> xyz=.10 .20 .85 rpy=-1.570796 0 3.141592
- joint joint_root: origin xyz=5.4 1.9 4.16 rpy=0 0 3.14159 -> xyz=.54 .19 .416 rpy=0 0 3.14159
- joint joint_tcp_1: origin xyz=-1.64 -0.28 2.32 -> xyz=-.164 -0.028 .232
- joint joint_tcp_2: origin xyz=-2.94 -0.11 0.44 rpy=0 -1.570796 0 -> xyz=-.294 -0.011 0.044 rpy=0 -1.570796 0
- joint kinect_depth_joint: origin xyz=5.15 9.6 14.55 rpy=0 0.87 -1.57 -> xyz=0.515 0.96 1.455 rpy=0 0.87 -1.57

Commit message: scale rollback

File: lbr3_model/lbr_gripper_pinch.urdf (robot description, URDF)
Before this commit: robot lbr3, 20 links, 19 joints
Links:
- link link_kinect: geometry visual box size=0.6 2.8 .4
- link segment_0: geometry collision mesh filename=package://lbr3_model/cad/segment_0_collision.dae scale=0.01 0.01 0.01; visual mesh filename=package://lbr3_model/cad/segment_0.dae scale=0.01 0.01 0.01
- link segment_1: geometry collision mesh filename=package://lbr3_model/cad/segment_1_collision.dae scale=0.01 0.01 0.01; visual mesh filename=package://lbr3_model/cad/segment_1.dae scale=0.01 0.01 0.01
- link segment_2: geometry collision mesh filename=package://lbr3_model/cad/segment_2_collision.dae scale=0.01 0.01 0.01; visual mesh filename=package://lbr3_model/cad/segment_2.dae scale=0.01 0.01 0.01
- link segment_3: geometry collision mesh filename=package://lbr3_model/cad/segment_3_collision.dae scale=0.01 0.01 0.01; visual mesh filename=package://lbr3_model/cad/segment_3.dae scale=0.01 0.01 0.01
- link segment_4: geometry collision mesh filename=package://lbr3_model/cad/segment_4_collision.dae scale=0.01 0.01 0.01; visual mesh filename=package://lbr3_model/cad/segment_4.dae scale=0.01 0.01 0.01
- link segment_5: geometry collision mesh filename=package://lbr3_model/cad/segment_5_collision.dae scale=0.01 0.01 0.01; visual mesh filename=package://lbr3_model/cad/segment_5.dae scale=0.01 0.01 0.01
- link segment_6: geometry collision mesh filename=package://lbr3_model/cad/segment_6_collision.dae scale=0.01 0.01 0.01; visual mesh filename=package://lbr3_model/cad/segment_6.dae scale=0.01 0.01 0.01
- link segment_7: geometry collision mesh filename=package://lbr3_model/cad/segment_7_collision.dae scale=0.01 0.01 0.01; visual mesh filename=package://lbr3_model/cad/segment_7.dae scale=0.01 0.01 0.01
- link tool: geometry collision mesh filename=package://kuka_description/cad/tool_s.dae; visual mesh filename=package://kuka_description/cad/tool_s.dae
Joints:
- joint joint_0: origin xyz=0 0 .1105 -> xyz=0 0 1.105
- joint joint_1: origin xyz=0 0 .2 -> xyz=0 0 2
- joint joint_2: origin xyz=0 0 .2 -> xyz=0 0 2
- joint joint_3: origin xyz=0 0 .2 -> xyz=0 0 2
- joint joint_4: origin xyz=0 0 .2 -> xyz=0 0 2
- joint joint_5: origin xyz=0 0 .1885 -> xyz=0 0 1.885
- joint joint_6: origin xyz=0 0 .0795 -> xyz=0 0 .795
- joint joint_goal_2: origin xyz=.20 .10 1.20 rpy=-1.570796 0 1.570796 -> xyz=2.0 1.0 12.0 rpy=-1.570796 0 1.570796
- joint joint_goal_3: origin xyz=.20 .15 1.20 rpy=-1.570796 0 1.570796 -> xyz=2.0 1.5 12.0 rpy=-1.570796 0 1.570796
- joint joint_goal_4: origin xyz=.20 .20 .85 rpy=-1.570796 0 3.141592 -> xyz=2.0 2.0 8.5 rpy=-1.570796 0 3.141592
- joint joint_goal_5: origin xyz=.15 .20 .85 rpy=-1.570796 0 3.141592 -> xyz=1.5 2.0 8.5 rpy=-1.570796 0 3.141592
- joint joint_goal_6: origin xyz=.10 .20 .85 rpy=-1.570796 0 3.141592 -> xyz=1.0 2.0 8.5 rpy=-1.570796 0 3.141592
- joint joint_root: origin xyz=.54 .19 .416 rpy=0 0 3.14159 -> xyz=5.4 1.9 4.16 rpy=0 0 3.14159
- joint joint_tcp_1: origin xyz=-.164 -0.028 .232 -> xyz=-1.64 -0.28 2.32
- joint joint_tcp_2: origin xyz=-.294 -0.011 0.044 rpy=0 -1.570796 0 -> xyz=-2.94 -0.11 0.44 rpy=0 -1.570796 0
- joint kinect_depth_joint: origin xyz=0.515 0.96 1.455 rpy=0 0.87 -1.57 -> xyz=5.15 9.6 14.55 rpy=0 0.87 -1.57

Commit message: move robot to center

File: lbr3_model/lbr_gripper_pinch.urdf (robot description, URDF)
Before this commit: robot lbr3, 20 links, 19 joints
Joints:
- joint joint_goal_1: origin xyz=2.0 0.5 12.0 rpy=-1.570796 0 1.570796 -> xyz=3.4 1.4 7.84 rpy=-1.570796 0 -1.570796
- joint joint_goal_2: origin xyz=2.0 1.0 12.0 rpy=-1.570796 0 1.570796 -> xyz=2.0 1.0 12.0 rpy=-1.570796 0 -1.570796
- joint joint_goal_3: origin xyz=2.0 1.5 12.0 rpy=-1.570796 0 1.570796 -> xyz=2.0 1.5 12.0 rpy=-1.570796 0 -1.570796
- joint joint_goal_4: origin xyz=2.0 2.0 8.5 rpy=-1.570796 0 3.141592 -> xyz=2.0 2.0 8.5 rpy=-1.570796 0 0
- joint joint_root: origin xyz=5.4 1.9 4.16 rpy=0 0 3.14159 -> xyz=0 0 0 rpy=0 0 0

Commit message: ICRA15 video setting

File: lbr3_model/lbr_gripper_pinch.urdf (robot description, URDF)
Before this commit: robot lbr3, 20 links, 19 joints
Joints:
- joint joint_goal_1: origin xyz=3.4 1.4 7.84 rpy=-1.570796 0 -1.570796 -> xyz=3.4 1.4 7.84 rpy=1.570796 0 1.570796

Commit message: video setting for gripper

File: lbr3_model/lbr_gripper_pinch.urdf (robot description, URDF)
Before this commit: robot lbr3, 20 links, 19 joints
Links:
- added link finger_1_link_0, mass 0.05; collision mesh filename=package://robotiq_s_model_visualization/meshes/s-model_arti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; visual mesh filename=package://robotiq_s_model_visualization/meshes/s-model_arti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
- added link finger_1_link_1, mass 0.15; collision mesh filename=package://robotiq_s_model_visualization/meshes/s-model_arti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; visual mesh filename=package://robotiq_s_model_visualization/meshes/s-model_arti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
- added link finger_1_link_2, mass 0.15; collision mesh filename=package://robotiq_s_model_visualization/meshes/s-model_arti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; visual mesh filename=package://robotiq_s_model_visualization/meshes/s-model_arti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
- added link finger_1_link_3, mass 0.05; collision mesh filename=package://robotiq_s_model_visualization/meshes/s-model_arti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; visual mesh filename=package://robotiq_s_model_visualization/meshes/s-model_arti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
- added link finger_2_link_0, mass 0.05; collision mesh filename=package://robotiq_s_model_visualization/meshes/s-model_arti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; visual mesh filename=package://robotiq_s_model_visualization/meshes/s-model_arti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
- added link finger_2_link_1, mass 0.15; collision mesh filename=package://robotiq_s_model_visualization/meshes/s-model_arti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; visual mesh filename=package://robotiq_s_model_visualization/meshes/s-model_arti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
- added link finger_2_link_2, mass 0.15; collision mesh filename=package://robotiq_s_model_visualization/meshes/s-model_arti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; visual mesh filename=package://robotiq_s_model_visualization/meshes/s-model_arti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
- added link finger_2_link_3, mass 0.05; collision mesh filename=package://robotiq_s_model_visualization/meshes/s-model_arti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; visual mesh filename=package://robotiq_s_model_visualization/meshes/s-model_arti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
- added link finger_middle_link_0, mass 0.05; collision mesh filename=package://robotiq_s_model_visualization/meshes/s-model_arti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; visual mesh filename=package://robotiq_s_model_visualization/meshes/s-model_arti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
- added link finger_middle_link_1, mass 0.15; collision mesh filename=package://robotiq_s_model_visualization/meshes/s-model_arti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; visual mesh filename=package://robotiq_s_model_visualization/meshes/s-model_arti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
- added link finger_middle_link_2, mass 0.15; collision mesh filename=package://robotiq_s_model_visualization/meshes/s-model_arti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; visual mesh filename=package://robotiq_s_model_visualization/meshes/s-model_arti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
- added link finger_middle_link_3, mass 0.05; collision mesh filename=package://robotiq_s_model_visualization/meshes/s-model_arti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; visual mesh filename=package://robotiq_s_model_visualization/meshes/s-model_arti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
- added link palm, mass 1.3; collision mesh filename=package://robotiq_s_model_visualization/meshes/s-model_arti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; visual mesh filename=package://robotiq_s_model_visualization/meshes/s-model_arti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
- added link tcp_3_link
- link link_kinect: geometry visual box size=0.06 .28 .04
- link segment_0: geometry collision mesh filename=package://lbr3_model/cad/segment_0_collision.dae scale=0.001 0.001 0.001; visual mesh filename=package://lbr3_model/cad/segment_0.dae scale=0.001 0.001 0.001
- link segment_1: geometry collision mesh filename=package://lbr3_model/cad/segment_1_collision.dae scale=0.001 0.001 0.001; visual mesh filename=package://lbr3_model/cad/segment_1.dae scale=0.001 0.001 0.001
- link segment_2: geometry collision mesh filename=package://lbr3_model/cad/segment_2_collision.dae scale=0.001 0.001 0.001; visual mesh filename=package://lbr3_model/cad/segment_2.dae scale=0.001 0.001 0.001
- link segment_3: geometry collision mesh filename=package://lbr3_model/cad/segment_3_collision.dae scale=0.001 0.001 0.001; visual mesh filename=package://lbr3_model/cad/segment_3.dae scale=0.001 0.001 0.001
- link segment_4: geometry collision mesh filename=package://lbr3_model/cad/segment_4_collision.dae scale=0.001 0.001 0.001; visual mesh filename=package://lbr3_model/cad/segment_4.dae scale=0.001 0.001 0.001
- link segment_5: geometry collision mesh filename=package://lbr3_model/cad/segment_5_collision.dae scale=0.001 0.001 0.001; visual mesh filename=package://lbr3_model/cad/segment_5.dae scale=0.001 0.001 0.001
- link segment_6: geometry collision mesh filename=package://lbr3_model/cad/segment_6_collision.dae scale=0.001 0.001 0.001; visual mesh filename=package://lbr3_model/cad/segment_6.dae scale=0.001 0.001 0.001
- link segment_7: geometry collision mesh filename=package://lbr3_model/cad/segment_7_collision.dae scale=0.001 0.001 0.001; visual mesh filename=package://lbr3_model/cad/segment_7.dae scale=0.001 0.001 0.001
- link tool: geometry 
Joints:
- added joint finger_1_joint_1: type revolute, parent finger_1_link_0, child finger_1_link_1, origin xyz=0.020 0 0 rpy=0 0 0, axis 0 0 1, limit lower=0 upper=3.1416 effort=100 velocity=100, mimic joint=finger_middle_joint_1 multiplier=1
- added joint finger_1_joint_2: type fixed, parent finger_1_link_1, child finger_1_link_2, origin xyz=0.050 -.028 0 rpy=0 0 -0.52, axis 0 0 1, limit lower=0 upper=3.1416 effort=100 velocity=100
- added joint finger_1_joint_3: type fixed, parent finger_1_link_2, child finger_1_link_3, origin xyz=0.039 0 0 rpy=0 0 -0.61, axis 0 0 1, limit lower=-1.0 upper=3.1416 effort=100 velocity=100
- added joint finger_2_joint_1: type revolute, parent finger_2_link_0, child finger_2_link_1, origin xyz=0.020 0 0 rpy=0 0 0, axis 0 0 1, limit lower=0 upper=3.1416 effort=100 velocity=100, mimic joint=finger_middle_joint_1 multiplier=1
- added joint finger_2_joint_2: type fixed, parent finger_2_link_1, child finger_2_link_2, origin xyz=0.050 -.028 0 rpy=0 0 -0.52, axis 0 0 1, limit lower=0 upper=3.1416 effort=100 velocity=100
- added joint finger_2_joint_3: type fixed, parent finger_2_link_2, child finger_2_link_3, origin xyz=0.039 0 0 rpy=0 0 -0.61, axis 0 0 1, limit lower=-1.0 upper=3.1416 effort=100 velocity=100
- added joint finger_middle_joint_1: type revolute, parent finger_middle_link_0, child finger_middle_link_1, origin xyz=0.020 0 0 rpy=0 0 0, axis 0 0 1, limit lower=0 upper=3.1416 effort=100 velocity=100
- added joint finger_middle_joint_2: type fixed, parent finger_middle_link_1, child finger_middle_link_2, origin xyz=0.050 -.028 0 rpy=0 0 -0.52, axis 0 0 1, limit lower=0 upper=3.1416 effort=100 velocity=100
- added joint finger_middle_joint_3: type fixed, parent finger_middle_link_2, child finger_middle_link_3, origin xyz=0.039 0 0 rpy=0 0 -0.5579, axis 0 0 1, limit lower=-1.0 upper=3.1416 effort=100 velocity=100
- added joint joint_tcp_3: type fixed, parent segment_7, child tcp_3_link, origin xyz=0 0 .25, axis 0 0 1
- added joint palm_finger_1_joint: type fixed, parent palm, child finger_1_link_0, origin xyz=-0.0455 0.0214 0.036 rpy=0 2.9816 -1.57, axis 0 1 0, limit lower=-0.16 upper=0.25 effort=100 velocity=100
- added joint palm_finger_2_joint: type fixed, parent palm, child finger_2_link_0, origin xyz=-0.0455 0.0214 -0.036 rpy=0 3.3016 -1.57, axis 0 1 0, limit lower=-0.25 upper=0.16 effort=100 velocity=100
- added joint palm_finger_middle_joint: type fixed, parent palm, child finger_middle_link_0, origin xyz=0.0455 0.0214 0 rpy=0 0 1.57, axis 0 0 1
- added joint wrist: type fixed, parent segment_7, child palm, origin xyz=0 0 0.05 rpy=1.57 0 2.9, axis 0 0 1
- joint joint_0: origin xyz=0 0 1.105 -> xyz=0 0 .1105
- joint joint_1: origin xyz=0 0 2 -> xyz=0 0 .2
- joint joint_2: origin xyz=0 0 2 -> xyz=0 0 .2
- joint joint_3: origin xyz=0 0 2 -> xyz=0 0 .2
- joint joint_4: origin xyz=0 0 2 -> xyz=0 0 .2
- joint joint_5: origin xyz=0 0 1.885 -> xyz=0 0 0.1885
- joint joint_6: origin xyz=0 0 .795 -> xyz=0 0 .0795
- joint joint_tcp_1: origin xyz=-1.64 -0.28 2.32 -> xyz=-.164 -.028 .232
- joint joint_tcp_2: origin xyz=-2.94 -0.11 0.44 rpy=0 -1.570796 0 -> xyz=-.294 -.011 .044 rpy=0 -1.570796 0
- joint kinect_depth_joint: origin xyz=5.15 9.6 14.55 rpy=0 0.87 -1.57 -> xyz=0.515 0.96 1.455 rpy=0 0.87 -1.57

Commit message: use scaled meshes for robot

File: lbr3_model/lbr_gripper_pinch.urdf (robot description, URDF)
Before this commit: robot lbr3, 34 links, 33 joints
Links:
- removed link finger_1_link_0
- removed link finger_1_link_1
- removed link finger_1_link_2
- removed link finger_1_link_3
- removed link finger_2_link_0
- removed link finger_2_link_1
- removed link finger_2_link_2
- removed link finger_2_link_3
- removed link finger_middle_link_0
- removed link finger_middle_link_1
- removed link finger_middle_link_2
- removed link finger_middle_link_3
- removed link kuka_root
- removed link palm
- link segment_0: geometry collision mesh filename=package://lbr3_model/cad/segment_0_collision_s.dae; visual mesh filename=package://lbr3_model/cad/segment_0.dae scale=0.001 0.001 0.001
- link segment_1: geometry collision mesh filename=package://lbr3_model/cad/segment_1_collision_s.dae; visual mesh filename=package://lbr3_model/cad/segment_1.dae scale=0.001 0.001 0.001
- link segment_2: geometry collision mesh filename=package://lbr3_model/cad/segment_2_collision_s.dae; visual mesh filename=package://lbr3_model/cad/segment_2.dae scale=0.001 0.001 0.001
- link segment_3: geometry collision mesh filename=package://lbr3_model/cad/segment_3_collision_s.dae; visual mesh filename=package://lbr3_model/cad/segment_3.dae scale=0.001 0.001 0.001
- link segment_4: geometry collision mesh filename=package://lbr3_model/cad/segment_4_collision_s.dae; visual mesh filename=package://lbr3_model/cad/segment_4.dae scale=0.001 0.001 0.001
- link segment_5: geometry collision mesh filename=package://lbr3_model/cad/segment_5_collision_s.dae; visual mesh filename=package://lbr3_model/cad/segment_5.dae scale=0.001 0.001 0.001
- link segment_6: geometry collision mesh filename=package://lbr3_model/cad/segment_6_collision_s.dae; visual mesh filename=package://lbr3_model/cad/segment_6.dae scale=0.001 0.001 0.001
- link segment_7: geometry collision mesh filename=package://lbr3_model/cad/segment_7_collision_s.dae; visual mesh filename=package://lbr3_model/cad/segment_7.dae scale=0.001 0.001 0.001
- link tool: geometry collision mesh filename=package://kuka_description/cad/tool_s.dae; visual mesh filename=package://kuka_description/cad/tool.dae scale=0.001 0.001 0.001
Joints:
- removed joint finger_1_joint_1
- removed joint finger_1_joint_2
- removed joint finger_1_joint_3
- removed joint finger_2_joint_1
- removed joint finger_2_joint_2
- removed joint finger_2_joint_3
- removed joint finger_middle_joint_1
- removed joint finger_middle_joint_2
- removed joint finger_middle_joint_3
- removed joint joint_root
- removed joint palm_finger_1_joint
- removed joint palm_finger_2_joint
- removed joint palm_finger_middle_joint
- removed joint wrist
- joint joint_goal_1: parent kuka_root -> segment_0
- joint joint_goal_2: origin xyz=2.0 1.0 12.0 rpy=-1.570796 0 -1.570796 -> xyz=2.0 1.0 12.0 rpy=0 -1.570796 3.141592; parent kuka_root -> segment_0
- joint joint_goal_3: parent kuka_root -> segment_0
- joint joint_goal_4: parent kuka_root -> segment_0
- joint joint_goal_5: parent kuka_root -> segment_0
- joint joint_goal_6: parent kuka_root -> segment_0

Commit message: render PRM graph

File: lbr3_model/lbr_gripper_pinch.urdf (robot description, URDF)
Before this commit: robot lbr3, 20 links, 19 joints
Links:
- added link segment_00; collision mesh filename=package://lbr3_model/cad/segment_0_collision_s.dae; visual mesh filename=package://lbr3_model/cad/segment_0.dae scale=0.001 0.001 0.001
- link segment_0: geometry 
Joints:
- added joint joint_segment_0: type fixed, parent segment_0, child segment_00, origin xyz=0.3 0 0, axis 0 0 1
- joint joint_0: parent segment_0 -> segment_00
